File: ESP32_Trainer/ESP32_Trainer.kicad_sch (KiCad schematic)
At the start: 29 parts, among them J1 I2C, J2 SPI, J3 I2C, J4 MOSFET, Q1 2N3904, Q2 IRFZ44N, SW1 Push, SW2 Push, U1 ESP32_DevKit_V1_DOIT

Commit message: Por si cambio
Parts:
- added D5: 1N4006, Diode_THT:D_DO-41_SOD81_P10.16mm_Horizontal, symbol Diode:1N4006
- added J5: MOSFET, TerminalBlock:TerminalBlock_bornier-2_P5.08mm, symbol Connector:Screw_Terminal_01x02
- added J6: I2C, Connector_PinHeader_2.54mm:PinHeader_1x04_P2.54mm_Vertical, symbol Connector_Generic:Conn_01x04
- added J7: Barrel_Jack_Switch, Connector_BarrelJack:BarrelJack_Horizontal, symbol Connector:Barrel_Jack_Switch
- added J8: Conn_01x05, Connector_PinHeader_2.54mm:PinHeader_1x05_P2.54mm_Vertical, symbol Connector_Generic:Conn_01x05
- added Q3: 2N3904, Package_TO_SOT_THT:TO-92L_Inline_Wide, symbol Transistor_BJT:2N3904
- added Q4: IRFZ44N, Package_TO_SOT_THT:TO-220-3_Vertical, symbol @EmersonPrez15:IRFZ44N
- added R10: 1K, Resistencias_0.25W:1K, symbol Device:R_Small
- added R11: 2.2K, Resistencias_0.25W:1K, symbol Device:R_Small
- added R12, R13, R14: 10K, Resistencias_0.25W:1K, symbol Device:R_Small
- added U2: LM7805_TO220, Package_TO_SOT_THT:TO-220-3_Horizontal_TabDown, symbol Regulator_Linear:LM7805_TO220
- R1, R2, R3, R4, R5, R6, R7, R8, R9: footprint Resistor_THT:R_Axial_DIN0207_L6.3mm_D2.5mm_P10.16mm_Horizontal -> Resistencias_0.25W:1K
Connections:
- net +3.3V: now also J6.2 (Pin_2), R13.1, R14.1
- net +5V: now also D5.1 (K), R12.1
- net GND: now also J6.1 (Pin_1), J7.2, J7.3, Q3.1 (E), Q4.3 (S), R11.2, U2.2 (GND)
- net LED_1: now also U1.10 (D27/GPIO27/ADC2/TOUCH7); no longer U1.8 (D25/GPIO25/ADC2/DAC1)
- net LED_2: now also U1.11 (D14/GPIO14/ADC2/TOUCH6); no longer U1.9 (D26/GPIO26/ADC2/DAC2)
- net LED_3: now also U1.12 (D12/GPIO12/ADC2/TOUCH5); no longer U1.10 (D27/GPIO27/ADC2/TOUCH7)
- net MOSFET: now also U1.8 (D25/GPIO25/ADC2/DAC1); no longer U1.22 (UART2TX/GPIO17/D17)
- net PUSH: now also U1.4 (D34/GPIO34/ADC1); no longer C2.1, R9.1, SW2.1
- net RX: now also J6.3 (Pin_3)
- net SCL: now also R13.2
- net SDA: now also R14.2
- net TX: now also J6.4 (Pin_4)
- net VCC: now also J5.1 (Pin_1), J7.1, U2.1 (VI)
- net TOUCH3/ADC15/GPIO15/D15: now reaches U1.18 (TOUCH3/ADC15/GPIO15/D15)
- net TOUCH3/ADC15/GPIO15/D15: now also J8.1 (Pin_1)
- net TOUCH2/ADC2/GPIO2/D2: now reaches U1.19 (TOUCH2/ADC2/GPIO2/D2)
- net TOUCH2/ADC2/GPIO2/D2: now also J8.2 (Pin_2)
- net TOUCH0/ADC2/GPIO4/D4: now reaches U1.20 (TOUCH0/ADC2/GPIO4/D4)
- net TOUCH0/ADC2/GPIO4/D4: now also J8.3 (Pin_3)
- net UART2RX/GPIO16/D16: now reaches U1.21 (UART2RX/GPIO16/D16)
- net UART2RX/GPIO16/D16: now also J8.4 (Pin_4)
- net PUSH_2: now reaches U1.5 (D35/GPIO35/ADC1)
- net PUSH_2: now also C2.1, R9.1, SW2.1
- new net: Q3.2 (B), R10.2, R11.1
- new net: D5.2 (A), U2.3 (VO)
- new net: Q3.3 (C), Q4.1 (G), R12.2
- new net: J5.2 (Pin_2), Q4.2 (D)
- new net MOSFET_2: R10.1, U1.9 (D26/GPIO26/ADC2/DAC2)
- new net UART2TX/GPIO17/D17: J8.5 (Pin_5), U1.22 (UART2TX/GPIO17/D17)
Other:
- moved on the sheet: RV1
