File: ESP32_Trainer/ESP32_Trainer.kicad_pcb (KiCad board)
At the start: 2 copper layers, 99.1 x 63.5 mm, 29 parts, among them J1 I2C, J2 SPI, J3 I2C, J4 MOSFET, Q1 2N3904, Q2 IRFZ44N, SW1 Push, SW2 Push, U1 ESP32_DevKit_V1_DOIT

Commit message: Por si cambio
Parts:
- added D5: 1N4006, Diode_THT:D_DO-41_SOD81_P10.16mm_Horizontal, F.Cu at (71.1, 74.3)
- added J5: MOSFET, TerminalBlock:TerminalBlock_bornier-2_P5.08mm, F.Cu at (121.9, 44.5)
- added J6: I2C, Connector_PinHeader_2.54mm:PinHeader_1x04_P2.54mm_Vertical, F.Cu at (132.1, 95.2)
- added J7: Barrel_Jack_Switch, Connector_BarrelJack:BarrelJack_Horizontal, F.Cu at (68.9, 58.4)
- added J8: Conn_01x05, Connector_PinHeader_2.54mm:PinHeader_1x05_P2.54mm_Vertical, F.Cu at (63.5, 113.0)
- added Q3: 2N3904, Package_TO_SOT_THT:TO-92L_Inline_Wide, F.Cu at (102.2, 49.5)
- added Q4: IRFZ44N, Package_TO_SOT_THT:TO-220-3_Vertical, F.Cu at (110.2, 44.5)
- added R10: 1K, Resistencias_0.25W:1K, F.Cu at (94.6, 51.0)
- added R11: 2.2K, Resistencias_0.25W:1K, F.Cu at (97.8, 43.0)
- added R12: 10K, Resistencias_0.25W:1K, F.Cu at (106.0, 43.0)
- added R13: 10K, Resistencias_0.25W:1K, F.Cu at (108.0, 82.2)
- added R14: 10K, Resistencias_0.25W:1K, F.Cu at (100.2, 82.2)
- added U2: LM7805_TO220, Package_TO_SOT_THT:TO-220-3_Horizontal_TabDown, F.Cu at (74.6, 76.8)
- R1, R2, R3, R4, R5, R6, R7, R8, R9: footprint Resistor_THT:R_Axial_DIN0207_L6.3mm_D2.5mm_P10.16mm_Horizontal -> Resistencias_0.25W:1K
- moved H1 171.4 mm to (64.4, 44.5)
- moved H3 165.7 mm to (73.7, 113.0)
- moved Q1 140.9 mm to (102.2, 63.0), turned to 90 degrees
- moved J1 139.8 mm to (95.9, 106.0), turned to 90 degrees
- moved J2 132.8 mm to (87.8, 106.0), turned to -90 degrees
- moved RV1 130.1 mm to (76.2, 63.0), turned to -90 degrees
- moved J3 129.3 mm to (111.1, 106.0), turned to 90 degrees
- moved J4 125.1 mm to (121.9, 58.4), turned to -90 degrees
- moved R4 124.9 mm to (94.6, 64.5), turned to 90 degrees
- moved R5 122.9 mm to (97.8, 56.5), turned to -90 degrees
- moved D4 116.9 mm to (127.6, 104.8)
- moved R6 115.4 mm to (106.0, 56.5), turned to -90 degrees
- moved Q2 107.5 mm to (110.2, 58.4), turned to -90 degrees
- moved H4 103.7 mm to (135.5, 112.8)
- moved H2 103.0 mm to (135.3, 42.3)
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Connections:
- C2 pad 1: PUSH -> PUSH_2
- R9 pad 1: PUSH -> PUSH_2
- SW2 pad 1: PUSH -> PUSH_2
- U1 pad 10: LED_3 -> LED_1
- U1 pad 11: unconnected-(U1-D14/GPIO14/ADC2/TOUCH6-Pad11) -> LED_2
- U1 pad 12: unconnected-(U1-D12/GPIO12/ADC2/TOUCH5-Pad12) -> LED_3
- U1 pad 18: unconnected-(U1-TOUCH3/ADC15/GPIO15/D15-Pad18) -> TOUCH3/ADC15/GPIO15/D15
- U1 pad 19: unconnected-(U1-TOUCH2/ADC2/GPIO2/D2-Pad19) -> TOUCH2/ADC2/GPIO2/D2
- U1 pad 20: unconnected-(U1-TOUCH0/ADC2/GPIO4/D4-Pad20) -> TOUCH0/ADC2/GPIO4/D4
- U1 pad 21: unconnected-(U1-UART2RX/GPIO16/D16-Pad21) -> UART2RX/GPIO16/D16
- U1 pad 22: MOSFET -> UART2TX/GPIO17/D17
- U1 pad 4: unconnected-(U1-D34/GPIO34/ADC1-Pad4) -> PUSH
- U1 pad 5: unconnected-(U1-D35/GPIO35/ADC1-Pad5) -> PUSH_2
- U1 pad 8: LED_1 -> MOSFET
- U1 pad 9: LED_2 -> MOSFET_2
Routing:
- net +3.3V: track 0.00 -> 246.2 mm, vias 0 -> 4
- net VCC: track 0.00 -> 123.4 mm
- net +5V: track 0.00 -> 103.2 mm, vias 0 -> 2
- net SCL: track 0.00 -> 68.7 mm
- net PUSH_2: track 0.00 -> 49.6 mm, vias 0 -> 2
- net UART2TX/GPIO17/D17: track 0.00 -> 49.0 mm
- net UART2RX/GPIO16/D16: track 0.00 -> 45.3 mm
- net SDA: track 0.00 -> 43.3 mm
- net TOUCH0/ADC2/GPIO4/D4: track 0.00 -> 42.0 mm
- net GND: track 0.00 -> 41.3 mm, vias 0 -> 10
- net TOUCH2/ADC2/GPIO2/D2: track 0.00 -> 38.7 mm
- net RX: track 0.00 -> 37.1 mm
- net PUSH: track 0.00 -> 36.2 mm
- net TOUCH3/ADC15/GPIO15/D15: track 0.00 -> 36.2 mm
- net TX: track 0.00 -> 29.4 mm
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- added copper zone on B.Cu, net GND
Other:
- board size 99.1 x 63.5 mm -> 80 x 80 mm

Commit message: Asistencia
Parts:
- added kibuzzard-6849B320: G***, kibuzzard-6849B320, F.Cu at (87.9, 101.5)
- added kibuzzard-6849B34F: G***, kibuzzard-6849B34F, F.Cu at (85.3, 101.5)
- added kibuzzard-6849B368: G***, kibuzzard-6849B368, F.Cu at (82.8, 101.4)
- added kibuzzard-6849B37B: G***, kibuzzard-6849B37B, F.Cu at (80.2, 102.7)
- added kibuzzard-6849B38C: G***, kibuzzard-6849B38C, F.Cu at (77.6, 101.7)
- added kibuzzard-6849B393: G***, kibuzzard-6849B393, F.Cu at (75.1, 101.8)
- added kibuzzard-6849B41C: G***, kibuzzard-6849B41C, F.Cu at (67.2, 102.9)
- added kibuzzard-6849B428: G***, kibuzzard-6849B428, F.Cu at (67.2, 105.4)
- added kibuzzard-6849B446: G***, kibuzzard-6849B446, F.Cu at (66.8, 107.9)
- added kibuzzard-6849B454: G***, kibuzzard-6849B454, F.Cu at (66.8, 110.5)
- added kibuzzard-6849B45E: G***, kibuzzard-6849B45E, F.Cu at (67.2, 113.0)
- added kibuzzard-6849B4B1: G***, kibuzzard-6849B4B1, F.Cu at (118.9, 110.4)
- added kibuzzard-6849B4B1: G***, kibuzzard-6849B4B1, F.Cu at (103.6, 110.2)
- added kibuzzard-6849B4BD: G***, kibuzzard-6849B4BD, F.Cu at (116.2, 110.6)
- added kibuzzard-6849B4BD: G***, kibuzzard-6849B4BD, F.Cu at (101.0, 110.4)
- added kibuzzard-6849B4C9: G***, kibuzzard-6849B4C9, F.Cu at (113.6, 110.2)
- added kibuzzard-6849B4C9: G***, kibuzzard-6849B4C9, F.Cu at (98.4, 110.0)
- added kibuzzard-6849B4D4: G***, kibuzzard-6849B4D4, F.Cu at (111.0, 110.3)
- added kibuzzard-6849B4D4: G***, kibuzzard-6849B4D4, F.Cu at (95.8, 110.1)
- added kibuzzard-6849B511: G***, kibuzzard-6849B511, F.Cu at (124.5, 91.8)
- added kibuzzard-6849B51A: G***, kibuzzard-6849B51A, F.Cu at (126.9, 91.8)
- added kibuzzard-6849B53A: G***, kibuzzard-6849B53A, F.Cu at (129.4, 91.8)
- added kibuzzard-6849B541: G***, kibuzzard-6849B541, F.Cu at (134.7, 95.1)
- added kibuzzard-6849B815: G***, kibuzzard-6849B815, F.Cu at (128.8, 44.3)
- added kibuzzard-6849B815: G***, kibuzzard-6849B815, F.Cu at (128.8, 58.2)
Routing:
- net +5V: track 103.2 -> 102.5 mm
