File: Proyectos_KiCad/ESP32_Trainer_38Pin/ESP32_Trainer_38Pin.kicad_sch (KiCad schematic)
At the start: 8 parts, among them J1 DC JACK, U1 LM7805_TO220

Commit message: Todo por si cambio
Parts:
- removed C2: 100nF, Capacitor_THT:C_Disc_D3.8mm_W2.6mm_P2.50mm, symbol Device:C_Small
- added C3: 100nF, PCM_Capacitor_THT_AKL:C_Disc_D3.8mm_W2.6mm_P2.50mm, symbol Device:C_Small
- added D4, D5: ~, LED_SMD:LED_1210_3225Metric_Pad1.42x2.65mm_HandSolder, symbol Device:LED_Small
- added H1, H2, H3, H4: ~, MountingHole:MountingHole_3.2mm_M3_Pad_Via, symbol Mechanical:MountingHole_Pad
- added J2: GPIO, PCM_SL_Connectors:PinHeader_1x04_P2.54mm_Vertical, symbol Connector_Generic:Conn_01x04
- added J3: SPI, PCM_SL_Connectors:PinHeader_1x06_P2.54mm_Vertical, symbol Connector_Generic:Conn_01x06
- added J4, J5: UART, PCM_SL_Connectors:PinHeader_1x04_P2.54mm_Vertical, symbol Connector_Generic:Conn_01x04
- added J6, J7: LOAD1, TerminalBlock_Phoenix:TerminalBlock_Phoenix_MKDS-1,5-2-5.08_1x02_P5.08mm_Horizontal, symbol Connector:Screw_Terminal_01x02
- added LED1: RGB, PCM_LED_THT_AKL:LED_D5.0mm-4_RGB_Wide_Pins, symbol PCM_LED_AKL:LED_5mm_RGB_Kcom_RKBG
- added Q1, Q2: 2N3904, PCM_Package_TO_SOT_SMD_AKL:SOT-23_BigPads, symbol Transistor_BJT:2N3904
- added Q3, Q4: BD139, Package_TO_SOT_THT:TO-126-3_Vertical, symbol Transistor_BJT:BD139
- added R1, R2: 470, Resistencias_0.25W:470, symbol Device:R_Small
- added R10, R9: 1K, PCM_Resistor_SMD_AKL:R_0805_2012Metric_Pad1.15x1.40mm_HandSolder, symbol Device:R_Small
- added R11, R12: 150, PCM_Resistor_SMD_AKL:R_0805_2012Metric_Pad1.15x1.40mm_HandSolder, symbol Device:R_Small
- added R13: 100, PCM_Resistor_SMD_AKL:R_0805_2012Metric_Pad1.15x1.40mm_HandSolder, symbol Device:R_Small
- added R4, R5: 10K, Resistencias_0.25W:10K, symbol Device:R_Small
- added R6, R7, R8: 470, PCM_Resistor_SMD_AKL:R_0805_2012Metric_Pad1.15x1.40mm_HandSolder, symbol Device:R_Small
- added RV1: 100K, PCM_Potentiometer_THT_AKL:Potentiometer_Bourns_3266Y_Vertical, symbol Device:R_Potentiometer
- added SW1, SW2: Push, Button_Switch_THT:SW_PUSH_6mm, symbol Switch:SW_Push
- added U2: ESP32-38pin, @EmersonPrez15:ESP32_DevKit_38Pin, symbol @EmersonPrez15:ESP32_DevKit_38Pin
- added U3: ~, @EmersonPrez15:SSD1306, symbol @EmersonPrez15:OLED_SSD1306
- C1: footprint Capacitor_THT:C_Disc_D3.8mm_W2.6mm_P2.50mm -> PCM_Capacitor_THT_AKL:C_Disc_D3.8mm_W2.6mm_P2.50mm
- D1: footprint LED_THT:LED_D5.0mm -> LED_SMD:LED_1210_3225Metric_Pad1.42x2.65mm_HandSolder
- D3: value LED_Small -> ~; footprint (none) -> LED_SMD:LED_1210_3225Metric_Pad1.42x2.65mm_HandSolder
- R3: renamed from R1; footprint Resistencias_0.25W:1K -> PCM_Resistor_SMD_AKL:R_0805_2012Metric_Pad1.15x1.40mm_HandSolder
- U1: footprint Package_TO_SOT_THT:TO-220-3_Vertical -> Package_TO_SOT_THT:TO-220-3_Horizontal_TabDown
Connections:
- net +5V: now also J2.1 (Pin_1), U2.19 (VIN/5V), U3.2 (VCC)
- net GND: now also D3.1 (K), C3.2, D4.1 (K), D5.1 (K), J2.2 (Pin_2), J3.6 (Pin_6), J4.1 (Pin_1), J5.1 (Pin_1), LED1.2 (A), Q3.1 (E), Q4.1 (E), R1.2, R2.2, RV1.3, U2.14 (GND), U2.32 (GND), U2.38 (GND), U3.1 (GND)
- net VCC: now also J6.1 (Pin_1), J7.1 (Pin_1); no longer C1.1
- net at D3.2 (A): now also R6.2
- new net: J6.2 (Pin_2), Q1.3 (C), Q3.2 (C)
- new net: LED1.4 (G), R12.2
- new net: Q2.1 (E), Q4.3 (B)
- new net: Q2.2 (B), R10.2
- new net: J7.2 (Pin_2), Q2.3 (C), Q4.2 (C)
- new net: LED1.1 (R), R13.2
- new net: D5.2 (A), R8.2
- new net: LED1.3 (B), R11.2
- new net: D4.2 (A), R7.2
- new net: Q1.2 (B), R9.2
- new net: Q1.1 (E), Q3.3 (B)
- new net +3.3V: J3.5 (Pin_5), J4.2 (Pin_2), J5.2 (Pin_2), R4.1, R5.1, RV1.1, SW1.2, SW2.2, U2.1 (3V3)
- new net BLUE: R12.1, U2.26 (TOU0/ADC2_0/GPIO4)
- new net CS: J3.4 (Pin_4), U2.29 (VSPI_CS/GPIO5)
- new net GPIO15: J2.3 (Pin_3), U2.23 (CS/TOU3/ADC2_3/GPIO15)
- new net GPIO2: J2.4 (Pin_4), U2.24 (TOU2/ADC2_2/GPIO2)
- new net GREEN: R11.1, U2.27 (RXD/GPIO16)
- new net LED1: R6.1, U2.13 (GPIO12/ADC2_5/TOU5/MISO)
- new net LED2: R7.1, U2.12 (GPIO14/ADC2_6/TOU6/CLK)
- new net LED3: R8.1, U2.11 (GPIO27/ADC2_7/TOU7)
- new net MISO: J3.2 (Pin_2), U2.31 (VSPI_MISO/GPIO19)
- new net MOSI: J3.1 (Pin_1), U2.37 (VSPI_MOSI/GPIO23)
- new net POT: RV1.2, U2.8 (GPIO33/ADC1_5/TOU8)
- new net PUSH_1: C1.1, R1.1, SW1.1, U2.5 (GPIO34/ADC1_6)
- new net PUSH_2: C3.1, R2.1, SW2.1, U2.6 (GPIO35/ADC1_7)
- new net PWM_1: R10.1, U2.10 (GPIO26/ADC2_9/DAC2)
- new net PWM_2: R9.1, U2.9 (GPIO25/ADC2_8/DAC1)
- new net RED: R13.1, U2.28 (TXD/GPIO17)
- new net RX: J4.3 (Pin_3), U2.34 (RXD/GPIO3)
- new net SCL: J5.3 (Pin_3), R4.2, U2.36 (SCL/GPIO22), U3.3 (SCL)
- new net SCLK: J3.3 (Pin_3), U2.30 (VSPI_CLK/GPIO18)
- new net SDA: J5.4 (Pin_4), R5.2, U2.33 (SDA/GPIO21), U3.4 (SDA)
- new net TX: J4.4 (Pin_4), U2.35 (TXD/GPIO1)
- no-connect marks 0 -> 12

Commit message: Placa entrenadora esp32-38
Parts:
- removed D1: ~, LED_SMD:LED_1210_3225Metric_Pad1.42x2.65mm_HandSolder, symbol Device:LED_Small
- removed R3: 1K, PCM_Resistor_SMD_AKL:R_0805_2012Metric_Pad1.15x1.40mm_HandSolder, symbol Device:R_Small
- D3, D4, D5: footprint LED_SMD:LED_1210_3225Metric_Pad1.42x2.65mm_HandSolder -> PCM_LED_THT_AKL:LED_D3.0mm
- R1, R2: footprint Resistencias_0.25W:470 -> PCM_Resistor_SMD_AKL:R_1206_3216Metric_Pad1.30x1.75mm_HandSolder
- R10, R11, R12, R13, R6, R7, R8, R9: footprint PCM_Resistor_SMD_AKL:R_0805_2012Metric_Pad1.15x1.40mm_HandSolder -> PCM_Resistor_SMD_AKL:R_1206_3216Metric_Pad1.42x1.75mm_HandSolder
Connections:
- net +3.3V: now also U3.2 (VCC)
- net +5V: no longer U3.2 (VCC)
- net PUSH_1: now also C3.1, R2.1, SW2.1; no longer C1.1, R1.1, SW1.1
- net PUSH_2: now also C1.1, R1.1, SW1.1; no longer C3.1, R2.1, SW2.1
- net PWM_1: now also R9.1; no longer R10.1
- net PWM_2: now also R10.1; no longer R9.1
- no-connect marks 12 -> 13
