File: Proyectos_KiCad/WS2812_NANO/WS2812_NANO.kicad_sch (KiCad schematic)
At the start: 0 parts

Commit message: WS2812 NANO
Parts:
- added A1: Arduino_Nano_Every, Module:Arduino_Nano, symbol MCU_Module:Arduino_Nano_Every
- added C1, C2: 100nF, Capacitor_THT:C_Disc_D3.8mm_W2.6mm_P2.50mm, symbol Device:C_Small
- added C3: 220uF, Capacitor_THT:CP_Radial_D5.0mm_P2.00mm, symbol Device:C_Polarized_Small
- added J1, J2: Conn_01x03, PCM_SL_Connectors:PinHeader_1x03_P2.54mm_Vertical, symbol Connector_Generic:Conn_01x03
- added J3: VLEDS, TerminalBlock_Phoenix:TerminalBlock_Phoenix_MKDS-1,5-2-5.08_1x02_P5.08mm_Horizontal, symbol Connector:Screw_Terminal_01x02
- added J4, J5: Conn_01x02, PCM_SL_Connectors:PinHeader_1x02_P2.54mm_Vertical, symbol Connector_Generic:Conn_01x02
- added R1, R2: 470, PCM_Resistor_SMD_AKL:R_1210_3225Metric_Pad1.30x2.65mm_HandSolder, symbol Device:R_Small
- added R3, R4: 220, Resistencias_0.25W:1K, symbol Device:R_Small
Connections:
- new net: A1.13 (D10), R3.2
- new net: A1.12 (D9), R4.2
- new net +5V: A1.27 (+5V), J4.1 (Pin_1), J5.1 (Pin_1)
- new net GND: A1.29 (GND), A1.4 (GND), C1.2, C2.2, C3.2, J1.3 (Pin_3), J2.3 (Pin_3), J3.2 (Pin_2), R1.2, R2.2
- new net POT: A1.22 (A3)
- new net PUSH_T1: A1.19 (A0), C2.1, J5.2 (Pin_2), R2.1
- new net PUSH_T2: A1.20 (A1), C1.1, J4.2 (Pin_2), R1.1
- new net T1: J1.2 (Pin_2), R3.1
- new net T2: J2.2 (Pin_2), R4.1
- new net VCC: C3.1, J1.1 (Pin_1), J2.1 (Pin_1), J3.1 (Pin_1)
