File: Proyectos_KiCad/Placa_Eddy/Placa_Eddy.kicad_sch (KiCad schematic)
At the start: 37 parts, among them J1 MOTOR_1, J10 TEMP2, J11 TEMP3, J12 TEMP4, J13 DC_JACK, J14 ON/OFF, J2 MOTOR_2, J3 MOTOR_3, J4 MOTOR_4, J5 TEMP1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

Commit message: Placa Eddy Terminada
Parts:
- removed J13: DC_JACK, symbol Connector:Barrel_Jack_Switch
- removed J14: ON/OFF, 4ms_Connector:Pins_1x02_2.54mm_TH, symbol PCM_4ms_Connector:Conn_01x02
- added J13: VC_MOTOR, TerminalBlock_Phoenix:TerminalBlock_Phoenix_MKDS-1,5-2_1x02_P5.00mm_Horizontal, symbol Connector:Screw_Terminal_01x02
- added J14: VC_S, TerminalBlock_Phoenix:TerminalBlock_Phoenix_MKDS-1,5-2_1x02_P5.00mm_Horizontal, symbol Connector:Screw_Terminal_01x02
- C1, C8: value 100uF/16V -> 100uF/25V; footprint (none) -> PCM_Capacitor_SMD_Handsoldering_AKL:CP_Elec_5x5.4
- C2, C3, C4, C5, C6, C7: footprint (none) -> PCM_Capacitor_SMD_Handsoldering_AKL:CP_Elec_5x5.4
- D1: footprint (none) -> LED_THT:LED_D5.0mm
- J1, J2, J3, J4: footprint 4ms_Connector:Pins_1x04_2.54mm_TH_SWD -> Connector_Molex:Molex_KK-254_AE-6410-04A_1x04_P2.54mm_Vertical
- J10, J11, J12, J9: footprint 4ms_Connector:Pins_1x03_2.54mm_TH_AudioInsRGndL -> Connector_Molex:Molex_KK-254_AE-6410-03A_1x03_P2.54mm_Vertical
- J5: value TEMP1 -> INF2; footprint 4ms_Connector:Pins_1x03_2.54mm_TH_AudioInsRGndL -> Connector_Molex:Molex_KK-254_AE-6410-03A_1x03_P2.54mm_Vertical
- J6: value TEMP1 -> INF1; footprint 4ms_Connector:Pins_1x03_2.54mm_TH_AudioInsRGndL -> Connector_Molex:Molex_KK-254_AE-6410-03A_1x03_P2.54mm_Vertical
- J7: value TEMP1 -> INF3; footprint 4ms_Connector:Pins_1x03_2.54mm_TH_AudioInsRGndL -> Connector_Molex:Molex_KK-254_AE-6410-03A_1x03_P2.54mm_Vertical
- J8: value TEMP1 -> INF4; footprint 4ms_Connector:Pins_1x03_2.54mm_TH_AudioInsRGndL -> Connector_Molex:Molex_KK-254_AE-6410-03A_1x03_P2.54mm_Vertical
- R1, R2, R3, R4, R5: footprint (none) -> PCM_Resistor_SMD_AKL:R_1206_3216Metric_Pad1.30x1.75mm
- U1: footprint Personal:esp32_devkit_v1_doit -> @EmersonPrez15:ESP32_DEVKIT_V1_E32
- U2, U4: footprint PCM_SL_Breakout_Boards:A4988_Breakout -> @EmersonPrez15:A4988
- U3, U5: footprint (none) -> @EmersonPrez15:D_TMC2209_Ca
- U6, U7, U8, U9: footprint (none) -> @EmersonPrez15:LM2596S
Connections:
- net DIR_M1: now also U1.22 (UART2TX/GPIO17/D17)
- net DIR_M2: now also U1.25 (MISO/GPIO19/D19)
- net DIR_M3: now also U1.9 (D26/GPIO26/ADC2/DAC2)
- net DIR_M4: now also U1.11 (D14/GPIO14/ADC2/TOUCH6)
- net EN_M1: now also U1.20 (TOUCH0/ADC2/GPIO4/D4)
- net EN_M2: now also U1.30 (MOSI/GPIO23/D23)
- net EN_M3: now also U1.10 (D27/GPIO27/ADC2/TOUCH7)
- net EN_M4: now also U1.13 (D13/GPIO13/ADC2/TOUCH4)
- net GND: now also J13.2 (Pin_2), J14.2 (Pin_2)
- net STEP_M1: now also U1.23 (CSO/GPIO5/D5)
- net STEP_M2: now also U1.24 (CLK/GPIO18/D18)
- net STEP_M3: now also U1.8 (D25/GPIO25/ADC2/DAC1)
- net STEP_M4: now also U1.12 (D12/GPIO12/ADC2/TOUCH5)
- net VCC: now also J14.1 (Pin_1); no longer R1.1, U7.1 (IN+), U8.1 (IN+)
- net INF1: now reaches U1.18 (TOUCH3/ADC15/GPIO15/D15)
- net INF1: now also J6.1 (Pin_1)
- net ST4: now reaches U1.19 (TOUCH2/ADC2/GPIO2/D2)
- net ST4: now also J12.3 (Pin_3), R5.1
- net INF2: now reaches U1.21 (UART2RX/GPIO16/D16)
- net INF2: now also J5.1 (Pin_1)
- net ST1: now reaches U1.26 (SDA/GPIO21/D21)
- net ST1: now also J9.3 (Pin_3), R2.1
- net ST2: now reaches U1.29 (SCL/GPIO22/D22)
- net ST2: now also J11.3 (Pin_3), R3.1
- net INF4: now reaches U1.5 (D35/GPIO35/ADC1)
- net INF4: now also J8.1 (Pin_1)
- net ST3: now reaches U1.6 (D32/GPIO32/ADC1/TOUCH9)
- net ST3: now also J10.3 (Pin_3), R4.1
- net INF3: now reaches U1.7 (D33/GPIO33/ADC1/TOUCH8)
- net INF3: now also J7.1 (Pin_1)
- removed net D0: J10.3 (Pin_3), J11.3 (Pin_3), J12.3 (Pin_3), J5.1 (Pin_1), J6.1 (Pin_1), J7.1 (Pin_1), J8.1 (Pin_1), J9.3 (Pin_3), R2.1, R3.1, R4.1, R5.1
- new net VCC_M: J13.1 (Pin_1), R1.1, U7.1 (IN+), U8.1 (IN+)
Other:
- moved on the sheet: J10, J12, R4, R5
