File: Proyectos_KiCad/Placa_Eddy/_autosave-Placa_Eddy.kicad_pcb (KiCad board)
At the start: 2 copper layers, 150 x 100 mm, 37 parts, among them J1 MOTOR_1, J10 TEMP2, J11 TEMP3, J12 TEMP4, J13 VC_MOTOR, J14 VC_S, J2 MOTOR_2, J3 MOTOR_3, J4 MOTOR_4, J5 INF2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

Commit message: Añadiendo Lagrimas
Routing:
- net GND: track 15.2 -> 22.6 mm
