File: Proyectos_KiCad/Shield_Brazo/Shield_Brazo.kicad_sch (KiCad schematic)
At the start: 3 parts, among them U1 TMC2209, U2 ESP32_DevKit_V1_DOIT, U3 A4988

Commit message: Placa Brazo
Parts:
- removed U1: TMC2209, symbol @EmersonPrez15:Driver_TMC2209
- removed U2: ESP32_DevKit_V1_DOIT, Personal:esp32_devkit_v1_doit, symbol @EmersonPrez15:ESP32_DevKit_MP
- removed U3: A4988, PCM_SL_Breakout_Boards:A4988_Breakout, symbol PCM_SL_Breakout_Boards:A4988
- added H1, H2, H3, H4: ~, MountingHole:MountingHole_3.2mm_M3_Pad_Via, symbol Mechanical:MountingHole_Pad
Other:
- added sheet Drivers_NEMA (Drivers_NEMA.kicad_sch)
- added sheet MCU (MCU.kicad_sch)
- added sheet Power (Power.kicad_sch)
- added sheet Servo (Servo.kicad_sch)
