File: Proyectos_KiCad/Fuente_Simetrica/Fuente_Simetrica.kicad_pcb (KiCad board)
At the start: 2 copper layers, 120.3 x 100 mm, 78 parts, among them J1 Transformador, J2 5V, J3 5V, J4 5V, J5 5V, J6 5V, J7 DHT11, U1 LM317AT, U11 ACS712, U2 LM337SP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

Commit message: Cambiando a Omarchy
Parts:
- added REF**: MountingHole_3.2mm_M3_Pad_Via, MountingHole:MountingHole_3.2mm_M3_Pad_Via, F.Cu at (130.8, 43.2)
- added REF**: MountingHole_3.2mm_M3_Pad_Via, MountingHole:MountingHole_3.2mm_M3_Pad_Via, F.Cu at (240.0, 43.2)
- added REF**: MountingHole_3.2mm_M3_Pad_Via, MountingHole:MountingHole_3.2mm_M3_Pad_Via, F.Cu at (241.3, 133.3)
- added REF**: MountingHole_3.2mm_M3_Pad_Via, MountingHole:MountingHole_3.2mm_M3_Pad_Via, F.Cu at (130.9, 133.3)
- D1, D2, D3, D4: footprint PCM_Diode_THT_AKL:D_DO-41_SOD81_P7.62mm_Horizontal -> Diode_THT:D_A-405_P10.16mm_Horizontal
- R2, R3: value 240 -> 12K
- moved D2 2.48 mm to (152.2, 81.7)
- moved D4 2.48 mm to (152.2, 85.6)
Routing:
- net VAC2: track 22.7 -> 18.6 mm
- net VAC: track 22.3 -> 24.4 mm
- net -VCC: track 138.1 -> 139.7 mm
- net DHT11_OUT: track 89.8 -> 91.0 mm
- net Net-(D7-K): track 54.8 -> 53.7 mm
- net VCC: track 227.7 -> 226.9 mm
Other:
- board text added: "-5V"
- board text added: "-VADJ"
- board text added: "3.3V"
- board text added: "5V"
- board text added: "VADJ"
