File: Proyectos_KiCad/Fuente_Simetrica/POSITE_POWER.kicad_sch (KiCad schematic)
At the start: 26 parts, among them U1 LM317AT, U3 LM7805CT, U5 AMS1117-3.3

Commit message: Cambiando a Omarchy
Parts:
- R2: value 240 -> 12K
Changed lines of the file:
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@@
 			)
 		)
-		(property "Value" "240"
+		(property "Value" "12K"
 			(at 69.596 57.15 0)
 			(effects
