File: Proyectos_KiCad/Fuente_Simetrica/POWER_AC.kicad_sch (KiCad schematic)
At the start: 11 parts, among them J1 Transformador

Commit message: Cambiando a Omarchy
Parts:
- D1, D2, D3, D4: footprint PCM_Diode_THT_AKL:D_DO-41_SOD81_P7.62mm_Horizontal -> Diode_THT:D_A-405_P10.16mm_Horizontal
Changed lines of the file:
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@@
 			)
 		)
-		(property "Footprint" "PCM_Diode_THT_AKL:D_DO-41_SOD81_P7.62mm_Horizontal"
+		(property "Footprint" "Diode_THT:D_A-405_P10.16mm_Horizontal"
 			(at 60.96 41.91 0)
 			(effects
@@
 			)
 		)
-		(property "Footprint" "PCM_Diode_THT_AKL:D_DO-41_SOD81_P7.62mm_Horizontal"
+		(property "Footprint" "Diode_THT:D_A-405_P10.16mm_Horizontal"
 			(at 60.96 52.07 0)
 			(effects
@@
 			)
 		)
-		(property "Footprint" "PCM_Diode_THT_AKL:D_DO-41_SOD81_P7.62mm_Horizontal"
+		(property "Footprint" "Diode_THT:D_A-405_P10.16mm_Horizontal"
 			(at 73.66 41.91 0)
 			(effects
@@
 			)
 		)
-		(property "Footprint" "PCM_Diode_THT_AKL:D_DO-41_SOD81_P7.62mm_Horizontal"
+		(property "Footprint" "Diode_THT:D_A-405_P10.16mm_Horizontal"
 			(at 73.66 52.07 0)
 			(effects
