File: Proyectos_KiCad/Fuente_Simetrica/VCC-_POWER.kicad_sch (KiCad schematic)
At the start: 20 parts, among them U2 LM337SP, U4 L7905ACV

Commit message: Cambiando a Omarchy
Parts:
- R3: value 240 -> 12K
Changed lines of the file:
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@@
 			)
 		)
-		(property "Value" "240"
+		(property "Value" "12K"
 			(at 76.708 36.83 0)
 			(effects
