File: Proyectos_KiCad/Fuente_Simetrica/Fuente_Simetrica.kicad_sch (KiCad schematic)
At the start: 0 parts

Commit message: Routeo Termiando
Other:
- added sheet CONN (CONN.kicad_sch)
- added sheet ESP32 (ESP32.kicad_sch)
- added sheet POWER_AC (POWER_AC.kicad_sch)
- added sheet VCC+_POWER (POSITE_POWER.kicad_sch)
- added sheet VCC-_POWER (VCC-_POWER.kicad_sch)
Changed lines of the file:
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@@
 	(generator_version "9.0")
 	(paper "A4")
+	(sheet
+		(at 78.74 137.16)
+		(size 12.7 3.81)
+		(exclude_from_sim no)
+		(in_bom yes)
+		(on_board yes)
+		(dnp no)
+		(fields_autoplaced yes)
+		(stroke
+			(width 0.1524)
+			(type solid)
+		)
+		(fill
+			(color 0 0 0 0.0000)
+		)
+		(property "Sheetname" "VCC+_POWER"
+			(at 78.74 136.4484 0)
+			(effects
+				(font
+					(size 1.27 1.27)
+				)
+				(justify left bottom)
+			)
+		)
+		(property "Sheetfile" "POSITE_POWER.kicad_sch"
+			(at 78.74 141.5546 0)
+			(effects
+				(font
+					(size 1.27 1.27)
+				)
+				(justify left top)
+			)
+		)
+		(instances
+			(project "Fuente_Simetrica"
+				(path "/a35a497b-08a2-425c-bfb2-859166f73d06"
+					(page "4")
+				)
+			)
+		)
+	)
+	(sheet
+		(at 36.83 105.41)
+		(size 12.7 11.43)
+		(exclude_from_sim no)
+		(in_bom yes)
+		(on_board yes)
+		(dnp no)
+		(fields_autoplaced yes)
+		(stroke
+			(width 0.1524)
+			(type solid)
+		)
+		(fill
+			(color 0 0 0 0.0000)
+		)
+		(property "Sheetname" "ESP32"
+			(at 36.83 104.6984 0)
+			(effects
+				(font
+					(size 1.27 1.27)
+				)
+				(justify left bottom)
+			)
+		)
+		(property "Sheetfile" "ESP32.kicad_sch"
+			(at 36.83 117.4246 0)
+			(effects
+				(font
+					(size 1.27 1.27)
+				)
+				(justify left top)
+			)
+		)
+		(instances
+			(project "Fuente_Simetrica"
+				(path "/a35a497b-08a2-425c-bfb2-859166f73d06"
+					(page "2")
+				)
+			)
+		)
+	)
+	(sheet
+		(at 129.54 106.68)
+		(size 12.7 3.81)
+		(exclude_from_sim no)
+		(in_bom yes)
+		(on_board yes)
+		(dnp no)
+		(fields_autoplaced yes)
+		(stroke
+			(width 0.1524)
+			(type solid)
+		)
+		(fill
+			(color 0 0 0 0.0000)
+		)
+		(property "Sheetname" "CONN"
+			(at 129.54 105.9684 0)
+			(effects
+				(font
+					(size 1.27 1.27)
+				)
+				(justify left bottom)
+			)
+		)
+		(property "Sheetfile" "CONN.kicad_sch"
+			(at 129.54 111.0746 0)
+			(effects
+				(font
+					(size 1.27 1.27)
+				)
+				(justify left top)
+			)
+		)
+		(instances
+			(project "Fuente_Simetrica"
+				(path "/a35a497b-08a2-425c-bfb2-859166f73d06"
+					(page "6")
+				)
+			)
+		)
+	)
+	(sheet
+		(at 128.27 133.35)
+		(size 12.7 19.05)
+		(exclude_from_sim no)
+		(in_bom yes)
+		(on_board yes)
+		(dnp no)
+		(fields_autoplaced yes)
+		(stroke
+			(width 0.1524)
+			(type solid)
+		)
+		(fill
+			(color 0 0 0 0.0000)
+		)
+		(property "Sheetname" "VCC-_POWER"
+			(at 128.27 132.6384 0)
+			(effects
+				(font
+					(size 1.27 1.27)
+				)
+				(justify left bottom)
+			)
+		)
+		(property "Sheetfile" "VCC-_POWER.kicad_sch"
+			(at 128.27 152.9846 0)
+			(effects
+				(font
+					(size 1.27 1.27)
+				)
+				(justify left top)
+			)
+		)
+		(instances
+			(project "Fuente_Simetrica"
+				(path "/a35a497b-08a2-425c-bfb2-859166f73d06"
+					(page "5")
+				)
+			)
+		)
+	)
+	(sheet
+		(at 74.93 110.49)
+		(size 12.7 3.81)
+		(exclude_from_sim no)
+		(in_bom yes)
+		(on_board yes)
+		(dnp no)
+		(fields_autoplaced yes)
+		(stroke
+			(width 0.1524)
+			(type solid)
+		)
+		(fill
+			(color 0 0 0 0.0000)
+		)
+		(property "Sheetname" "POWER_AC"
+			(at 74.93 109.7784 0)
+			(effects
+				(font
+					(size 1.27 1.27)
+				)
+				(justify left bottom)
+			)
+		)
+		(property "Sheetfile" "POWER_AC.kicad_sch"
+			(at 74.93 114.8846 0)
+			(effects
+				(font
+					(size 1.27 1.27)
+				)
+				(justify left top)
+			)
+		)
+		(instances
+			(project "Fuente_Simetrica"
+				(path "/a35a497b-08a2-425c-bfb2-859166f73d06"
+					(page "3")
+				)
+			)
+		)
+	)
 	(sheet_instances
 		(path "/"

Commit message: Por si valgo
Changed lines of the file:
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@@
 	(paper "A4")
 	(sheet
-		(at 78.74 137.16)
-		(size 12.7 3.81)
+		(at 74.93 128.27)
+		(size 19.05 16.51)
 		(exclude_from_sim no)
 		(in_bom yes)
@@
 		)
 		(property "Sheetname" "VCC+_POWER"
-			(at 78.74 136.4484 0)
+			(at 74.93 127.5584 0)
 			(effects
 				(font
@@
 		)
 		(property "Sheetfile" "POSITE_POWER.kicad_sch"
-			(at 78.74 141.5546 0)
+			(at 74.93 145.3646 0)
 			(effects
 				(font
@@
 	)
 	(sheet
-		(at 129.54 106.68)
-		(size 12.7 3.81)
+		(at 110.49 96.52)
+		(size 12.7 15.24)
 		(exclude_from_sim no)
 		(in_bom yes)
@@
 		)
 		(property "Sheetname" "CONN"
-			(at 129.54 105.9684 0)
+			(at 110.49 95.8084 0)
 			(effects
 				(font
@@
 		)
 		(property "Sheetfile" "CONN.kicad_sch"
-			(at 129.54 111.0746 0)
+			(at 110.49 112.3446 0)
 			(effects
 				(font
@@
 	)
 	(sheet
-		(at 128.27 133.35)
+		(at 109.22 125.73)
 		(size 12.7 19.05)
 		(exclude_from_sim no)
@@
 		)
 		(property "Sheetname" "VCC-_POWER"
-			(at 128.27 132.6384 0)
+			(at 109.22 125.0184 0)
 			(effects
 				(font
@@
 		)
 		(property "Sheetfile" "VCC-_POWER.kicad_sch"
-			(at 128.27 152.9846 0)
+			(at 109.22 145.3646 0)
 			(effects
 				(font
@@
 	)
 	(sheet
-		(at 74.93 110.49)
-		(size 12.7 3.81)
+		(at 74.93 96.52)
+		(size 19.05 22.86)
 		(exclude_from_sim no)
 		(in_bom yes)
@@
 		)
 		(property "Sheetname" "POWER_AC"
-			(at 74.93 109.7784 0)
+			(at 74.93 95.8084 0)
 			(effects
 				(font
@@
 		)
 		(property "Sheetfile" "POWER_AC.kicad_sch"
-			(at 74.93 114.8846 0)
+			(at 74.93 119.9646 0)
 			(effects
 				(font
