File: Proyectos_KiCad/MaxESP_M/Drivers.kicad_sch (KiCad schematic)
At the start: 17 parts, among them J10 RJ45, J11 RJ45, J12 RJ45, J13 RJ45, U5 TMC2209, U6 TMC2209, U7 TMC2209, U8 TMC2209

Commit message: Por si valgo
Parts:
- R14, R15, R16: footprint PCM_Resistor_SMD_AKL:R_1206_3216Metric_Pad1.30x1.75mm -> PCM_Resistor_SMD_AKL:R_0805_2012Metric_Pad1.20x1.40mm_HandSolder
