File: Proyectos_KiCad/MaxESP_M/MaxESP_M.kicad_sch (KiCad schematic)
At the start: 0 parts

Commit message: Por si valgo
Other:
- sheet Drivers ports: added DIR1, DIR2, DIR34, EN, RXTMC, STP1, STP2, STP3, STP4, TXTMC; removed none
- sheet ESP32S ports: added AUX3, AUX4, AUX7, AUX8, DE+, DE-, DIR1, DIR2, DIR34, EN, ESP32_RST, PEC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; removed none
- sheet Misc: file untitled.kicad_sch -> Misc.kicad_sch
- sheet Misc ports: added AUX3, AUX4, AUX7, AUX8, DE+, DE-, PEC, RA+, RA-, RX0, RX2, SCL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; removed none
