File: Proyectos_KiCad/MaxESP_M/Power.kicad_sch (KiCad schematic)
At the start: 13 parts, among them J1 DC, J14 VOL SEL, J2 ON/OFF, U2 LM7805CT, U3 L7812CV

Commit message: Por si valgo
Parts:
- C2, C3, C4, C5, C6, C7, C8: footprint PCM_Capacitor_SMD_Handsoldering_AKL:C_1206_3216Metric_Pad1.33x1.80mm -> PCM_Capacitor_SMD_Handsoldering_AKL:C_0805_2012Metric_Pad1.18x1.45mm
Changed lines of the file:
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@@
 			)
 		)
-		(property "Footprint" "PCM_Capacitor_SMD_Handsoldering_AKL:C_1206_3216Metric_Pad1.33x1.80mm"
+		(property "Footprint" "PCM_Capacitor_SMD_Handsoldering_AKL:C_0805_2012Metric_Pad1.18x1.45mm"
 			(at 96.52 77.47 0)
 			(effects
@@
 			)
 		)
-		(property "Footprint" "PCM_Capacitor_SMD_Handsoldering_AKL:C_1206_3216Metric_Pad1.33x1.80mm"
+		(property "Footprint" "PCM_Capacitor_SMD_Handsoldering_AKL:C_0805_2012Metric_Pad1.18x1.45mm"
 			(at 128.27 77.47 0)
 			(effects
@@
 			)
 		)
-		(property "Footprint" "PCM_Capacitor_SMD_Handsoldering_AKL:C_1206_3216Metric_Pad1.33x1.80mm"
+		(property "Footprint" "PCM_Capacitor_SMD_Handsoldering_AKL:C_0805_2012Metric_Pad1.18x1.45mm"
 			(at 54.61 77.47 0)
 			(effects
@@
 			)
 		)
-		(property "Footprint" "PCM_Capacitor_SMD_Handsoldering_AKL:C_1206_3216Metric_Pad1.33x1.80mm"
+		(property "Footprint" "PCM_Capacitor_SMD_Handsoldering_AKL:C_0805_2012Metric_Pad1.18x1.45mm"
 			(at 27.94 76.2 0)
 			(effects
@@
 			)
 		)
-		(property "Footprint" "PCM_Capacitor_SMD_Handsoldering_AKL:C_1206_3216Metric_Pad1.33x1.80mm"
+		(property "Footprint" "PCM_Capacitor_SMD_Handsoldering_AKL:C_0805_2012Metric_Pad1.18x1.45mm"
 			(at 107.95 38.1 0)
 			(effects
@@
 			)
 		)
-		(property "Footprint" "PCM_Capacitor_SMD_Handsoldering_AKL:C_1206_3216Metric_Pad1.33x1.80mm"
+		(property "Footprint" "PCM_Capacitor_SMD_Handsoldering_AKL:C_0805_2012Metric_Pad1.18x1.45mm"
 			(at 139.7 77.47 0)
 			(effects
@@
 			)
 		)
-		(property "Footprint" "PCM_Capacitor_SMD_Handsoldering_AKL:C_1206_3216Metric_Pad1.33x1.80mm"
+		(property "Footprint" "PCM_Capacitor_SMD_Handsoldering_AKL:C_0805_2012Metric_Pad1.18x1.45mm"
 			(at 68.58 76.2 0)
 			(effects
