File: Proyectos_KiCad/ESP32_Trainer_V2.0/ESP32_Trainer_V2.0.kicad_pcb (KiCad board)
At the start: 2 copper layers, 61 parts, among them J1 VIM, J10 LOAD, J2 RELE, J3 I2C, J4 UART, J5 SPI, J6 PINES, J7 PINES, J8 POWER, J9 LOAD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

Commit message: Placa Entrenadora V2
Parts:
- removed JP1, JP4: ENABLE VIM, PCM_SL_Connectors:PinHeader_1x03_P2.54mm_Vertical
- added G***: NAME_20X4mm, @EmersonPrez15:NAME_20X4mm, F.Cu at (132.2, 113.8)
- D1, D2, D3, D4, Q1, Q2, Q3, Q5, R1, R10, R11, R13, R2, R3, R4, R5, R6, R7, R8, R9, U2: moved to B.Cu
- D7: footprint PCM_Diode_THT_AKL:D_DO-41_SOD81_P7.62mm_Horizontal -> PCM_Diode_SMD_AKL:D_SMA_BigPads; moved to B.Cu
- Q4, Q6: value IRFZ44N -> BD139; footprint PCM_Package_TO_SOT_THT_AKL:TO-220-3_Vertical_GDS -> PCM_Package_TO_SOT_THT_AKL:TO-126-3_Vertical_ECB
- R12, R14: value 10K -> 1K; moved to B.Cu
- moved RV1 129.2 mm to (81.3, 63.5)
- moved LED1 121.5 mm to (71.1, 63.5), turned to 180 degrees
- moved R2 118.7 mm to (62.2, 71.1), turned to 90 degrees
- moved J7 117.4 mm to (62.2, 107.3)
- moved H1 117.2 mm to (54.6, 54.6)
- moved R10 116.5 mm to (92.1, 66.0), turned to 180 degrees
- moved R3 116.3 mm to (64.8, 71.1), turned to 90 degrees
- moved R4 114.0 mm to (67.3, 71.1), turned to 90 degrees
- moved H4 109.3 mm to (54.0, 116.2)
- moved SW2 108.4 mm to (94.0, 56.5), turned to -90 degrees
- moved R9 107.6 mm to (100.3, 66.0), turned to 180 degrees
- moved R12 103.0 mm to (83.8, 95.5), turned to 90 degrees
- moved J5 102.6 mm to (68.6, 116.2), turned to 90 degrees
- moved C5 99.8 mm to (54.4, 75.6), turned to -90 degrees
- moved SW1 96.6 mm to (102.9, 56.5), turned to -90 degrees
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Connections:
- J3 pad 1: GND -> /ESP32/SDA
- J3 pad 2: +3.3V -> /ESP32/SCL
- J3 pad 3: /Pin_Header/SCL -> +3.3V
- J3 pad 4: /Pin_Header/SDA -> GND
- J4 pad 3: /Pin_Header/UART0TX -> /ESP32/UART0TX
- J4 pad 4: /Pin_Header/UART0RX -> /ESP32/UART0RX
- J5 pad 3: /Pin_Header/SLK -> /ESP32/CLK
- J5 pad 4: /Pin_Header/MISO -> /ESP32/MISO
- J5 pad 5: /Pin_Header/MOSI -> /ESP32/MOSI
- J5 pad 6: /Pin_Header/CS -> /ESP32/CS
- J6 pad 1: /Pin_Header/GPIO34 -> /ESP32/GPIO34
- J6 pad 2: /Pin_Header/GPIO35 -> /ESP32/GPIO35
- J6 pad 3: /Pin_Header/GPIO32 -> /ESP32/GPIO32
- J7 pad 1: /Pin_Header/GPIO2 -> /ESP32/GPIO2
- J7 pad 2: /Pin_Header/GPIO4 -> /ESP32/GPIO4
- J7 pad 3: /Pin_Header/GPIO16 -> /ESP32/GPIO16
- J7 pad 4: /Pin_Header/GPIO17 -> /ESP32/GPIO17
- JP2 pad 2: Net-(JP1-B) -> Net-(J9-Pin_1)
- JP3 pad 2: Net-(JP3-C) -> Net-(J10-Pin_1)
- Q3 pad 1: GND -> Net-(Q3-E)
- Q3 pad 3: Net-(Q3-C) -> Net-(J9-Pin_2)
- Q4 pad 1: Net-(Q3-C) -> GND
- Q4 pad 2: Net-(J9-Pin_2) -> Net-(J10-Pin_2)
- Q4 pad 3: GND -> Net-(Q4-B)
- Q5 pad 1: GND -> Net-(Q4-B)
- Q5 pad 3: Net-(Q5-C) -> Net-(J10-Pin_2)
- Q6 pad 1: Net-(Q5-C) -> GND
- Q6 pad 2: Net-(J10-Pin_2) -> Net-(J9-Pin_2)
- Q6 pad 3: GND -> Net-(Q3-E)
- R10 pad 2: /GPIO_IN/GPIO_IN_DI_2 -> /ESP32/GPIO_IN_DI_2
- R11 pad 1: /GPIO_OUT/GPIO_PWM_1 -> /ESP32/GPIO_PWM_1
- R12 pad 1: Net-(Q3-C) -> /ESP32/SDA
- R12 pad 2: +5V -> +3.3V
- R13 pad 1: /GPIO_OUT/GPIO_PWM_2 -> /ESP32/GPIO_PWM_2
- R14 pad 1: Net-(Q5-C) -> /ESP32/SCL
- R14 pad 2: +5V -> +3.3V
- R2 pad 1: /GPIO_OUT/LED_R -> /ESP32/LED_R
- R3 pad 1: /GPIO_OUT/LED_G -> /ESP32/LED_G
- R4 pad 1: /GPIO_OUT/LED_B -> /ESP32/LED_B
- R5 pad 1: /GPIO_OUT/GPIO_RELE -> /ESP32/GPIO_RELE
- R7 pad 1: /GPIO_OUT/GPIO_BUZZER -> /ESP32/GPIO_BUZZER
- R9 pad 2: /GPIO_IN/GPIO_IN_DI_1 -> /ESP32/GPIO_IN_DI_1
- RV1 pad 2: /GPIO_IN/GPIO_IN_AN -> /ESP32/GPIO_IN_AN
- SW1 pad 2: /GPIO_IN/GPIO_IN_DI_1 -> /ESP32/GPIO_IN_DI_1
- SW2 pad 2: /GPIO_IN/GPIO_IN_DI_2 -> /ESP32/GPIO_IN_DI_2
- U5 pad 3: /Pin_Header/SCL -> /ESP32/SCL
- U5 pad 4: /Pin_Header/SDA -> /ESP32/SDA
Routing:
- net +5V: track 0.00 -> 237.8 mm, vias 0 -> 10
- net +3.3V: track 0.00 -> 187.0 mm, vias 0 -> 6
- net +12V: track 0.00 -> 179.0 mm
- net /ESP32/GPIO_BUZZER: track 0.00 -> 93.6 mm, vias 0 -> 6
- net /ESP32/GPIO_PWM_1: track 0.00 -> 73.1 mm, vias 0 -> 2
- net GND: track 0.00 -> 72.2 mm, vias 0 -> 18
- net /ESP32/GPIO_PWM_2: track 0.00 -> 64.7 mm, vias 0 -> 2
- net /ESP32/GPIO_RELE: track 0.00 -> 52.7 mm
- net /ESP32/SDA: track 0.00 -> 46.8 mm
- net /ESP32/SCL: track 0.00 -> 37.9 mm
- net /ESP32/MOSI: track 0.00 -> 33.7 mm, vias 0 -> 2
- net /ESP32/GPIO_IN_DI_1: track 0.00 -> 31.4 mm
- net /ESP32/GPIO32: track 0.00 -> 28.0 mm
- net /ESP32/GPIO_IN_AN: track 0.00 -> 25.5 mm
- net COM: track 0.00 -> 24.8 mm
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- added copper zone on B.Cu, net GND
Other:
- board outline added: 100 x 70 mm
- board text added: "+12V"
- board text added: "+3.3V"
- board text added: "+5V"
- board text added: "3.3"
- board text added: "CL"
- board text added: "CS"
- board text added: "D12"
- board text added: "D13"
- board text added: "D14"
- board text added: "D15"
- board text added: "D16"
- board text added: "D17"
- board text added: "D2"
- board text added: "D25"
- board text added: "D26"
- board text added: "D27"
- board text added: "D32"
- board text added: "D33"
- board text added: "D34"
- board text added: "D35"
- board text added: "D36"
- board text added: "D39"
- board text added: "D4"
- board text added: "GND"
- board text added: "MI"
- board text added: "MO"
- board text added: "RX"
- board text added: "SCL"
- board text added: "SDA"
- board text added: "SEL"
- board text added: "TX"
