File: Proyectos_KiCad/ESP32_Trainer_V2.0/ESP32.kicad_sch (KiCad schematic)
At the start: 2 parts, among them U3 ESP32_DevKit_V1_DOIT

Commit message: Placa Entrenadora V2
Parts:
- added R12, R14: 10K, PCM_Resistor_SMD_AKL:R_0805_2012Metric_Pad1.15x1.40mm, symbol Device:R_Small
Connections:
- net SCL: now also R14.1
- net SDA: now also R12.1
- new net +3.3V: R12.2, R14.2
