File: Proyectos_KiCad/ESP32_Trainer_V2.0/ESP32_Trainer_V2.0.kicad_sch (KiCad schematic)
At the start: 0 parts

Commit message: Placa Entrenadora V2
Other:
- sheet ESP32 ports: added +5V, CLK, CS, GND, GPIO16, GPIO17, GPIO2, GPIO32, GPIO34, GPIO35, GPIO4, GPIO_BUZZER, GPIO_IN_AN, GPIO_IN_DI_1, GPIO_IN_DI_2, GPIO_PWM_1, GPIO_PWM_2, GPIO_RELE, LED_B, LED_G, LED_R, MISO, MOSI, SCL, SDA, UART0RX, UART0TX; removed none
- sheet GPIO_IN ports: added GPIO_IN_AN, GPIO_IN_DI_1, GPIO_IN_DI_2; removed none
- sheet GPIO_OUT ports: added GPIO_BUZZER, GPIO_PWM_1, GPIO_PWM_2, GPIO_RELE, LED_B, LED_G, LED_R; removed none
- sheet Pin_Header ports: added CS, GPIO16, GPIO17, GPIO2, GPIO32, GPIO34, GPIO35, GPIO4, MISO, MOSI, SCL, SDA, SLK, UART0RX, UART0TX; removed none
- sheet Power ports: added +5V, GND; removed none
