File: Proyectos_KiCad/ESP32_Trainer_V2.0/Pin_Header.kicad_sch (KiCad schematic)
At the start: 11 parts, among them J3 I2C, J4 UART, J5 SPI, J6 PINES, J7 PINES, J8 POWER, U5 SSD1306

Commit message: Placa Entrenadora V2
Connections:
- net +3.3V: now also J3.3 (Pin_3); no longer J3.2 (Pin_2)
- net GND: now also J3.4 (Pin_4); no longer J3.1 (Pin_1)
- net SCL: now also J3.2 (Pin_2); no longer J3.3 (Pin_3)
- net SDA: now also J3.1 (Pin_1); no longer J3.4 (Pin_4)
Other:
- moved on the sheet: J3
Changed lines of the file:
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@@
 	(wire
 		(pts
-			(xy 66.04 33.02) (xy 66.04 35.56)
-		)
-		(stroke
-			(width 0)
-			(type default)
-		)
-	)
-	(wire
-		(pts
-			(xy 60.96 33.02) (xy 60.96 36.83)
-		)
-		(stroke
-			(width 0)
-			(type default)
-		)
-	)
-	(wire
-		(pts
-			(xy 63.5 33.02) (xy 63.5 39.37)
+			(xy 66.04 29.21) (xy 66.04 35.56)
 		)
 		(stroke
@@
 	(wire
 		(pts
-			(xy 68.58 33.02) (xy 68.58 35.56)
-		)
-		(stroke
-			(width 0)
-			(type default)
-		)
-	)
-	(wire
-		(pts
 			(xy 99.06 33.02) (xy 99.06 35.56)
 		)
@@
 	(wire
 		(pts
+			(xy 68.58 29.21) (xy 68.58 35.56)
+		)
+		(stroke
+			(width 0)
+			(type default)
+		)
+	)
+	(wire
+		(pts
 			(xy 154.94 33.02) (xy 154.94 39.37)
 		)
@@
 	(wire
 		(pts
+			(xy 60.96 29.21) (xy 60.96 36.83)
+		)
+		(stroke
+			(width 0)
+			(type default)
+		)
+	)
+	(wire
+		(pts
 			(xy 41.91 35.56) (xy 41.91 38.1)
 		)
@@
 		(pts
 			(xy 144.78 36.83) (xy 144.78 33.02)
+		)
+		(stroke
+			(width 0)
+			(type default)
+		)
+	)
+	(wire
+		(pts
+			(xy 63.5 29.21) (xy 63.5 39.37)
 		)
 		(stroke
@@
 	(symbol
 		(lib_id "Connector_Generic:Conn_01x04")
-		(at 63.5 27.94 90)
+		(at 66.04 24.13 270)
+		(mirror x)
 		(unit 1)
 		(exclude_from_sim no)
@@
 		(on_board yes)
 		(dnp no)
-		(fields_autoplaced yes)
 		(property "Reference" "J3"
-			(at 64.77 21.59 90)
+			(at 64.77 17.78 90)
 			(effects
 				(font
@@
 		)
 		(property "Value" "I2C"
-			(at 64.77 24.13 90)
+			(at 64.77 20.32 90)
 			(effects
 				(font
@@
 		)
 		(property "Footprint" "Connector_PinHeader_2.54mm:PinHeader_1x04_P2.54mm_Horizontal"
-			(at 63.5 27.94 0)
+			(at 66.04 24.13 0)
 			(effects
 				(font
@@
 		)
 		(property "Datasheet" "~"
-			(at 63.5 27.94 0)
+			(at 66.04 24.13 0)
 			(effects
 				(font
@@
 		)
 		(property "Description" "Generic connector, single row, 01x04, script generated (kicad-library-utils/schlib/autogen/connector/)"
-			(at 63.5 27.94 0)
-			(effects
-				(font
+			(at 66.04 24.13 0)
+			(effects
+				(font
