File: Proyectos_KiCad/ULN2803R/ULN2803R.kicad_sch (KiCad schematic)
At the start: 9 parts, among them J1 IN, J2 OUT, J3 CARGADOR, J4 RELES, U1 ULN2803A

Commit message: Shiel-ULN2803-BPM
Parts:
- added U2: 74LS14, Package_DIP:CERDIP-14_W7.62mm_SideBrazed_LongPads, symbol 74xx:74LS14
- H1, H2, H3, H4: value ~ -> (none)
Connections:
- net GND: now also U2.7 (GND)
- net VCC: now also U2.14 (VCC)
- net at J1.1 (Pin_1): now also U2.9; no longer U1.6 (I6)
- net at J1.2 (Pin_2): now also U2.11; no longer U1.5 (I5)
- net at J1.3 (Pin_3): now also U2.5; no longer U1.4 (I4)
- net at J1.4 (Pin_4): now also U2.3; no longer U1.3 (I3)
- net at J1.5 (Pin_5): now also U2.1; no longer U1.2 (I2)
- new net: U1.3 (I3), U2.4
- new net: U1.5 (I5), U2.10
- new net: U1.4 (I4), U2.6
- new net: U1.2 (I2), U2.2
- new net: U1.6 (I6), U2.8
Other:
- moved on the sheet: J1
