File: Proyectos_KiCad/AguaV1.0/ESP32.kicad_sch (KiCad schematic)
At the start: 8 parts, among them J2 SSD1306, U1 ESP32_DevKit_V1_DOIT

Commit message: Omarchy-RIP
Parts:
- H1, H2, H3, H4: value ~ -> (none)
