File: Proyectos_KiCad/Caja-ESP32/Caja-ESP32.kicad_pcb (KiCad board)
At the start: 2 copper layers, 85 parts, among them J1 JACK_DC, J10 LOAD, J11 LOAD, J12 LOAD, J13 LOAD, J14 LOAD, J2 Fichero, J3 LOAD, J7 LOAD, J8 LOAD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

Commit message: Router
Parts:
- removed J11, J13, J9: LOAD, TerminalBlock_Phoenix:TerminalBlock_Phoenix_MKDS-1,5-2-5.08_1x02_P5.08mm_Horizontal
- added REF**: HT_9X15X20mm, @EmersonPrez15:HT_9X15X20mm, F.Cu at (67.5, 119.3)
- added REF**: HT_9X15X20mm, @EmersonPrez15:HT_9X15X20mm, F.Cu at (199.9, 60.1)
- added REF**: HT_9X15X20mm, @EmersonPrez15:HT_9X15X20mm, F.Cu at (200.0, 78.6)
- added REF**: HT_9X15X20mm, @EmersonPrez15:HT_9X15X20mm, F.Cu at (200.1, 116.2)
- added REF**: HT_9X15X20mm, @EmersonPrez15:HT_9X15X20mm, F.Cu at (200.0, 97.3)
- R18, R19, R22, R23, R26, R27, R28, R29: footprint Resistor_THT:R_Axial_DIN0207_L6.3mm_D2.5mm_P15.24mm_Horizontal -> Resistor_THT:R_Axial_DIN0207_L6.3mm_D2.5mm_P10.16mm_Horizontal
- U2: moved to B.Cu
- U6, U7, U8, U9: footprint Package_DIP:DIP-6_W7.62mm_LongPads -> @EmersonPrez15:MOC3020
- moved J7 136.9 mm to (228.6, 55.3), turned to 180 degrees
- moved J8 135.4 mm to (225.8, 65.2), turned to -90 degrees
- moved H2 133.8 mm to (193.0, 55.2)
- moved Q2 131.2 mm to (204.5, 65.1), turned to -90 degrees
- moved C7 127.7 mm to (214.1, 71.4), turned to 90 degrees
- moved Q3 125.9 mm to (204.8, 83.6), turned to -90 degrees
- moved R20 122.3 mm to (175.7, 65.1)
- moved C8 122.1 mm to (214.0, 89.8), turned to 90 degrees
- moved Q4 121.3 mm to (204.8, 102.3), turned to -90 degrees
- moved C2 120.2 mm to (87.5, 53.0), turned to -90 degrees
- moved Q5 117.9 mm to (204.8, 121.1), turned to -90 degrees
- moved C9 117.5 mm to (214.0, 108.5), turned to 90 degrees
- moved R21 116.0 mm to (175.8, 83.6)
- moved C10 114.1 mm to (214.0, 127.2), turned to 90 degrees
- moved J10 113.1 mm to (225.8, 83.6), turned to -90 degrees
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Connections:
- J10 pad 1: Net-(J10-Pin_1) -> AC_2
- J12 pad 1: Net-(J11-Pin_2) -> AC_2
- J14 pad 1: Net-(J13-Pin_2) -> AC_2
- J7 pad 1: Net-(J7-Pin_1) -> AC_2
- J7 pad 2: Net-(J7-Pin_2) -> AC_1
- J8 pad 1: Net-(J7-Pin_2) -> AC_2
- Q2 pad 2: Net-(J7-Pin_1) -> AC_1
- Q3 pad 2: Net-(J9-Pin_1) -> AC_1
- Q4 pad 2: Net-(J11-Pin_1) -> AC_1
- Q5 pad 2: Net-(J13-Pin_1) -> AC_1
- R18 pad 2: Net-(J7-Pin_1) -> AC_1
- R19 pad 2: Net-(J7-Pin_1) -> AC_1
- R22 pad 2: Net-(J9-Pin_1) -> AC_1
- R23 pad 2: Net-(J9-Pin_1) -> AC_1
- R26 pad 2: Net-(J11-Pin_1) -> AC_1
- R27 pad 2: Net-(J13-Pin_1) -> AC_1
- R28 pad 2: Net-(J11-Pin_1) -> AC_1
- R29 pad 2: Net-(J13-Pin_1) -> AC_1
- U1 pad 1: (no net) -> VCC
- U1 pad 2: (no net) -> GND
- U1 pad 3: (no net) -> Net-(D9-A)
- U1 pad 4: (no net) -> GND
- U10 pad 20: RELE_1 -> RELE_4
- U10 pad 21: RELE_2 -> unconnected-(U10-UART2RX/GPIO16/D16-Pad21)
- U10 pad 23: unconnected-(U10-CSO/GPIO5/D5-Pad23) -> RELE_2
- U10 pad 24: RELE_4 -> RELE_1
Routing:
- net +3.3V: track 0.00 -> 303.7 mm, vias 0 -> 6
- net AC_1: track 0.00 -> 195.8 mm
- net VCC: track 0.00 -> 131.3 mm
- net AC_2: track 0.00 -> 108.5 mm
- net IN_1: track 0.00 -> 103.6 mm, vias 0 -> 2
- net +5V: track 0.00 -> 98.8 mm, vias 0 -> 6
- net RELE_DC: track 0.00 -> 84.2 mm, vias 0 -> 2
- net BT_2: track 0.00 -> 66.6 mm
- net SCL: track 0.00 -> 60.3 mm
- net BT_3: track 0.00 -> 58.4 mm
- net SW_1: track 0.00 -> 58.2 mm
- net BT_1: track 0.00 -> 57.7 mm
- net SW_4: track 0.00 -> 57.6 mm, vias 0 -> 2
- net SDA: track 0.00 -> 56.1 mm
- net RELE_4: track 0.00 -> 56.1 mm
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- added copper zone on B.Cu, net GND
Other:
- board outline added: 198 x 83 mm
- board text added: "12V"
- board text added: "BT1"
- board text added: "BT2"
- board text added: "BT3"
- board text added: "GND"
- board text added: "LOAD"
- board text added: "OUTPUT TIP122"
- board text added: "VAC"

Commit message: Hola
Routing:
- net AC_1: track 195.8 -> 194.9 mm
