File: Proyectos_KiCad/Dispensador_Garrafones_V2.0/Dispensador_Garrafones_V2.0.kicad_pcb (KiCad board)
At the start: 2 copper layers, 230 x 90 mm, 93 parts, among them J1 JACK_DC, J10 LOAD, J11 FICHERO, J5 LOAD, J6 LOAD, J7 LOAD, J8 LOAD, J9 LOAD, Q1 TIP122, Q2 BT136-800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

Commit message: Nuevos Proyectos
Parts:
- added G***: LOGO, @EmersonPrez15:Dis, F.Cu at (179.1, 127.8)
- added G***: LOGO, @EmersonPrez15:CARITA_8x8mm, F.Cu at (193.8, 113.3)
- C3, C4, C5: footprint Capacitor_THT:C_Disc_D3.8mm_W2.6mm_P2.50mm -> Capacitor_THT:C_Disc_D4.3mm_W1.9mm_P5.00mm
- Q1, Q2, Q3, Q4, Q5: footprint Package_TO_SOT_THT:TO-220-3_Vertical -> @EmersonPrez15:TO-220-3_VDC
- R15, R18, R22, R23: footprint PCM_Resistor_THT_AKL:R_Axial_DIN0207_L6.3mm_D2.5mm_P15.24mm_Horizontal -> Resistor_THT:R_Axial_DIN0207_L6.3mm_D2.5mm_P10.16mm_Horizontal
- moved Q1 376.1 mm to (78.7, 120.1), turned to 90 degrees
- moved D4 371.4 mm to (69.8, 111.8), turned to -90 degrees
- moved JP1 363.7 mm to (68.6, 97.8)
- moved J11 359.5 mm to (62.2, 97.8), turned to -90 degrees
- moved R26 358.2 mm to (66.8, 90.9), turned to 180 degrees
- moved R12 358.0 mm to (83.3, 121.4), turned to 90 degrees
- moved R11 355.3 mm to (86.4, 121.4), turned to 90 degrees
- moved R10 352.5 mm to (89.7, 121.4), turned to 90 degrees
- moved Q6 352.5 mm to (79.5, 99.8), turned to 180 degrees
- moved U11 351.1 mm to (69.3, 90.9)
- moved J5 350.4 mm to (62.0, 115.1), turned to -90 degrees
- moved D3 349.2 mm to (83.3, 130.8), turned to 90 degrees
- moved U3 349.2 mm to (92.7, 121.4), turned to 90 degrees
- moved R28 346.1 mm to (80.0, 87.6), turned to -90 degrees
- moved R29 344.3 mm to (80.8, 104.1), turned to 180 degrees
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Connections:
- D4 pad 1: VCC -> +12V
- J1 pad 1: VCC -> +12V
- J10 pad 1: ADC2 -> ADC1
- J10 pad 2: ADC1 -> ADC2
- J5 pad 1: VCC -> +12V
- U1 pad 1: VCC -> +12V
- U3 pad 4: VCC -> +12V
- U8 pad 11: /Microcontrolador/RELE_4 -> /Microcontrolador/RELE_1
- U8 pad 4: /Microcontrolador/RELE_1 -> /Microcontrolador/RELE_4
- U8 pad 5: /Microcontrolador/RELE_2 -> /Microcontrolador/RELE_3
- U8 pad 6: /Microcontrolador/RELE_3 -> /Microcontrolador/RELE_2
Routing:
- net +5V: track 0.00 -> 306.7 mm, vias 0 -> 6
- net ADC1: track 0.00 -> 230.0 mm
- net +12V: track 0.00 -> 133.7 mm
- net /Microcontrolador/R_DIGITAL: track 0.00 -> 126.9 mm, vias 0 -> 4
- net ADC2: track 0.00 -> 102.8 mm
- net /Inputs/IN_FI: track 0.00 -> 96.2 mm, vias 0 -> 4
- net /Inputs/BT_1: track 0.00 -> 93.4 mm, vias 0 -> 2
- net +3.3V: track 0.00 -> 88.2 mm, vias 0 -> 4
- net SCL: track 0.00 -> 84.5 mm, vias 0 -> 2
- net SDA: track 0.00 -> 79.7 mm, vias 0 -> 2
- net /Inputs/SW_1: track 0.00 -> 67.8 mm
- net /ESP01/OUT_AR0: track 0.00 -> 66.5 mm, vias 0 -> 2
- net /Inputs/BT_2: track 0.00 -> 65.8 mm, vias 0 -> 2
- net /Inputs/SW_2: track 0.00 -> 63.3 mm
- net /Inputs/SW_3: track 0.00 -> 58.9 mm
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- added copper zone on B.Cu, net GND
Other:
- board size 230 x 90 mm -> 200 x 90 mm
- board text added: "+12V"
- board text added: "---"
- board text added: "BT1"
- board text added: "BT2"
- board text added: "BT3"
- board text added: "DIRECT"
- board text added: "GND"
- board text added: "IN"
- board text added: "IN AC"
- board text added: "LOAD"
- board text added: "OPTO"
- board text added: "RELE1"
- board text added: "RELE2"
- board text added: "RELE3"
- board text added: "RELE4"
- board text added: "RESET"
- board text added: "SW1"
- board text added: "SW2"
- board text added: "SW3"
- board text added: "SW4"
- board text added: "SW5"
