File: Proyectos_KiCad/Dispensador_Garrafones_V2.0/Dispensador_Garrafones_V2.0.kicad_pcb (KiCad board)
At the start: 2 copper layers, 200 x 90 mm, 95 parts, among them J1 JACK_DC, J10 LOAD, J11 FICHERO, J5 LOAD, J6 LOAD, J7 LOAD, J8 LOAD, J9 LOAD, Q1 TIP122, Q2 BT136-800, Q3 BT136-800, Q4 BT136-800, Q5 BT136-800, Q6 2N3906, SW1 SW_DIP_x05, SW2 Push_Button, U1 MP1584, U11 PC817, U12 PC817, U13 PC817, U2 AMS1117-3.3, U3 PC817, U4 MOC3021M, U5 MOC3021M, U6 MOC3021M, U7 MOC3021M, U8 Atmega328P-PU, U9 ESP-01S, Y1 Crystal_16MHz

Commit message: Modificaciones GarrV2
Parts:
- C6, C7, C8, C9: value C -> 10nF/400V
- J10, J6, J7, J8, J9: footprint TerminalBlock_Phoenix:TerminalBlock_Phoenix_MKDS-1,5-2-5.08_1x02_P5.08mm_Horizontal -> Connector_AMASS:AMASS_XT30U-F_1x02_P5.0mm_Vertical
- Q2, Q3, Q4, Q5: footprint @EmersonPrez15:TO-220-3_VDC -> PCM_Package_TO_SOT_THT_AKL:TO-3P-3_Vertical
- moved D6 14.1 mm to (198.1, 67.9), turned to -90 degrees
- moved D8 13.7 mm to (197.5, 114.3), turned to -90 degrees
- moved D7 13.2 mm to (197.5, 92.7), turned to -90 degrees
- moved D5 13.2 mm to (197.5, 47.0), turned to -90 degrees
- moved G*** 9.65 mm to (184.2, 113.3)
- moved R13 5.08 mm to (190.0, 60.5)
- moved R15 5.08 mm to (205.2, 51.6)
- moved R17 5.08 mm to (190.0, 106.2)
- moved R18 5.08 mm to (205.2, 73.2)
- moved R20 5.08 mm to (190.0, 82.0)
- moved R21 5.08 mm to (190.0, 129.0)
- moved R22 5.08 mm to (205.2, 97.3)
- moved R23 5.08 mm to (205.2, 119.4)
- moved U4 5.08 mm to (193.8, 54.1)
- moved U5 5.08 mm to (193.8, 99.8)
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Connections:
- U1 pad 1: +12V -> GND
- U1 pad 2: GND -> +12V
- U1 pad 3: Net-(D1-A) -> GND
- U1 pad 4: GND -> Net-(D1-A)
Routing:
- net ADC1: track 230.0 -> 258.6 mm
- net GND: track 11.1 -> 36.5 mm
- net +12V: track 133.7 -> 113.1 mm
- net Net-(D6-A): track 9.42 -> 23.7 mm
- net Net-(Q2-G): track 9.53 -> 23.8 mm
- net Net-(D8-A): track 9.41 -> 21.9 mm
- net Net-(D5-A): track 9.42 -> 21.9 mm
- net Net-(D7-A): track 9.42 -> 21.1 mm
- net Net-(D1-A): track 6.28 -> 13.7 mm
- net Net-(Q4-G): track 9.53 -> 16.2 mm
- net /Microcontrolador/RELE_1: track 58.8 -> 52.2 mm
- net Net-(Q5-G): track 9.53 -> 16.1 mm
- net Net-(Q3-G): track 9.53 -> 16.1 mm
- net /Microcontrolador/RELE_3: track 47.0 -> 42.1 mm
- net Net-(J8-Pin_2): track 36.3 -> 31.4 mm
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
Commit message: mejora
Connections:
- U9 pad 2: GPIO1 -> unconnected-(U9-GPIO1-Pad2)
- U9 pad 8: unconnected-(U9-TX-Pad8) -> GPIO1
Routing:
- net GPIO1: track 29.0 -> 25.6 mm

Commit message: Backup antes de reinstalacion del SO: proyectos y librerias KiCad
Parts:
- moved Q4 45.7 mm to (180.3, 67.0)
- moved Q1 45.3 mm to (180.4, 21.4)
- moved Q3 45.3 mm to (180.5, 42.9)
- moved Q5 45.3 mm to (180.7, 89.2)
- moved C5 45.0 mm to (197.1, 78.7)
- moved R16 45.0 mm to (191.3, 81.2)
- moved J5 45.0 mm to (207.3, 76.2)
- moved R13 44.8 mm to (156.2, 99.7)
- moved R14 44.6 mm to (171.1, 68.5)
- moved U6 44.6 mm to (159.6, 71.1)
- moved R12 44.6 mm to (155.8, 77.4)
- moved D5 44.6 mm to (163.3, 64.0)
- moved D4 44.5 mm to (163.5, 39.9)
- moved R34 44.5 mm to (100.3, 38.2)
- moved R18 44.5 mm to (32.8, 62.3)
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- renumbered C10 to C1, C1 to C10, C2 to C11, C11 to C2, C6 to C3, C7 to C4, C8 to C5, C9 to C6, C3 to C7, C4 to C8, C5 to C9, D5 to D1, D3 to D2, D4 to D3, D6 to D4, D7 to D5, D8 to D6, D9 to D7, D1 to D8, D2 to D9, J10 to J1, J3 to J10, J1 to J11, J7 to J2, J5 to J3, J8 to J4, J6 to J5, J9 to J6, J11 to J7, J2 to J8, J4 to J9, Q2 to Q1, Q1 to Q2, R34 to R1, R18 to R10, R19 to R11, R17 to R12, R21 to R13, R22 to R14, R23 to R15, R24 to R16, R25 to R17, R26 to R18, R4 to R19, R9 to R2, R5 to R20, R6 to R21, R7 to R22, R8 to R23, R28 to R24, R27 to R25, R29 to R26, R2 to R27, R14 to R28, R3 to R29, R13 to R3, R1 to R30, R30 to R31, R31 to R33, R33 to R34, R10 to R4, R15 to R5, R11 to R6, R12 to R7, R16 to R8, R20 to R9, SW2 to SW1, SW1 to SW2, U8 to U1, U2 to U10, U12 to U11, U13 to U12, U9 to U13, U10 to U2, U6 to U5, U5 to U6, U11 to U8, U1 to U9
Connections:
- C1 pad 1: Net-(U8-PB6_XTAL1) -> (no net)
- C2 pad 1: Net-(U8-PB7_XTAL2) -> (no net)
- C3 pad 1: Net-(C6-Pad1) (its old number) -> (no net)
- C3 pad 2: Net-(J7-Pin_2) (its old number) -> (no net)
- C4 pad 1: Net-(C7-Pad1) -> (no net)
- C4 pad 2: Net-(J8-Pin_2) -> (no net)
- C5 pad 1: Net-(C8-Pad1) -> (no net)
- C5 pad 2: Net-(J6-Pin_2) (its old number) -> (no net)
- J2 pad 2: Net-(J7-Pin_2) (its old number) -> Net-(J2-Pin_2)
- J4 pad 2: Net-(J8-Pin_2) -> Net-(J4-Pin_2)
- J5 pad 2: Net-(J6-Pin_2) (its old number) -> Net-(J5-Pin_2)
- Q1 pad 1: Net-(J7-Pin_2) (its old number) -> Net-(J2-Pin_2)
- Q1 pad 3: Net-(Q2-G) -> (no net)
- Q2 pad 1: Net-(Q1-B) -> (no net)
- Q3 pad 1: Net-(J8-Pin_2) -> Net-(J4-Pin_2)
- Q4 pad 1: Net-(J6-Pin_2) (its old number) -> Net-(J5-Pin_2)
- R1 pad 1: Net-(U8-PC6_RESET) -> (no net)
- R11 pad 1: Net-(C7-Pad1) -> Net-(C4-Pad1)
- R12 pad 2: Net-(R17-Pad2) -> (no net)
- R14 pad 1: Net-(R22-Pad1) -> (no net)
- R16 pad 1: Net-(C8-Pad1) -> Net-(C5-Pad1)
- R2 pad 2: Net-(R9-Pad2) (its old number) -> (no net)
- R24 pad 1: Net-(R27-Pad1) -> (no net)
- R25 pad 1: Net-(R27-Pad1) -> Net-(R24-Pad1)
- R3 pad 2: Net-(R13-Pad2) (its old number) -> (no net)
- R31 pad 2: Net-(R30-Pad2) -> (no net)
- R4 pad 1: Net-(R10-Pad1) (its old number) -> (no net)
- R4 pad 2: Net-(Q1-B) -> Net-(Q2-B)
- R5 pad 1: Net-(R15-Pad1) (its old number) -> (no net)
- R6 pad 2: Net-(Q1-B) -> Net-(Q2-B)
- R7 pad 2: Net-(Q1-B) -> Net-(Q2-B)
- R8 pad 1: Net-(C6-Pad1) (its old number) -> Net-(C3-Pad1)
- SW1 pad 2: Net-(U8-PC6_RESET) -> Net-(U1-PC6_RESET)
- U1 pad 1: Net-(U8-PC6_RESET) -> Net-(U1-PC6_RESET)
- U1 pad 10: Net-(U8-PB7_XTAL2) -> Net-(U1-PB7_XTAL2)
- U1 pad 2: unconnected-(U8-PD0_RXD-Pad2) -> (no net)
- U1 pad 3: unconnected-(U8-PD1_TXD-Pad3) -> (no net)
- U1 pad 9: Net-(U8-PB6_XTAL1) -> Net-(U1-PB6_XTAL1)
- U11 pad 1: Net-(R30-Pad2) -> Net-(R31-Pad2)
- U13 pad 2: unconnected-(U9-GPIO1-Pad2) -> GPIO1
- U13 pad 4: unconnected-(U9-RX-Pad4) -> (no net)
- U13 pad 6: unconnected-(U9-RST-Pad6) -> (no net)
- U13 pad 7: unconnected-(U9-CH-Pad7) -> (no net)
- U13 pad 8: GPIO1 -> (no net)
- U3 pad 1: Net-(R9-Pad2) (its old number) -> Net-(R2-Pad2)
- U3 pad 3: Net-(R10-Pad1) (its old number) -> Net-(R4-Pad1)
- U4 pad 1: Net-(R13-Pad2) (its old number) -> Net-(R3-Pad2)
- U4 pad 4: Net-(Q2-G) -> Net-(Q1-G)
- U4 pad 6: Net-(R15-Pad1) (its old number) -> Net-(R5-Pad1)
- U6 pad 1: Net-(R17-Pad2) -> Net-(R12-Pad2)
- U6 pad 6: Net-(R22-Pad1) -> Net-(R14-Pad1)
- U8 pad 4: Net-(R27-Pad1) -> Net-(R24-Pad1)
- Y1 pad 1: Net-(U8-PB6_XTAL1) -> Net-(U1-PB6_XTAL1)
- Y1 pad 2: Net-(U8-PB7_XTAL2) -> Net-(U1-PB7_XTAL2)
Routing:
- net Net-(J2-Pin_2): track 0.00 -> 35.6 mm
- net Net-(J5-Pin_2): track 0.00 -> 32.7 mm
- net Net-(J4-Pin_2): track 0.00 -> 32.6 mm
- net Net-(J7-Pin_2) (its old number): track 32.5 -> 0.00 mm
- net Net-(J8-Pin_2): track 31.4 -> 0.00 mm
- net Net-(J6-Pin_2) (its old number): track 31.2 -> 0.00 mm
- net Net-(Q2-G): track 23.8 -> 0.00 mm
- net Net-(Q1-G): track 0.00 -> 23.8 mm
- net Net-(U8-PC6_RESET): track 23.5 -> 0.00 mm
- net Net-(U1-PC6_RESET): track 0.00 -> 23.5 mm
- net Net-(Q2-B): track 0.00 -> 19.7 mm
- net Net-(Q1-B): track 19.7 -> 0.00 mm
- net Net-(R4-Pad1): track 0.00 -> 12.0 mm
- net Net-(R10-Pad1) (its old number): track 12.0 -> 0.00 mm
- net Net-(U8-PB6_XTAL1): track 10.1 -> 0.00 mm
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
Commit message: Guardar cambios generales
Parts:
- moved C5 0.43 mm to (197.5, 78.9)
- moved J5 0.43 mm to (207.6, 76.4)
- moved U6 0.43 mm to (160.0, 71.3)
- moved D5 0.43 mm to (163.7, 64.2)
- moved Q4 0.43 mm to (180.7, 67.2)
- moved R12 0.43 mm to (156.2, 77.7)
- moved R14 0.43 mm to (171.4, 68.8)
- moved R16 0.43 mm to (191.6, 81.5)
- moved C6 0.07 mm to (197.5, 101.0)
- moved J6 0.07 mm to (207.6, 98.5)
- moved R13 0.07 mm to (156.2, 99.8)
- moved U7 0.07 mm to (160.0, 93.4)
- moved D6 0.07 mm to (163.7, 86.3)
- moved Q5 0.07 mm to (180.7, 89.3)
- moved R15 0.07 mm to (171.4, 90.9)
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Connections:
- C1 pad 1: (no net) -> Net-(U1-PB6_XTAL1)
- C2 pad 1: (no net) -> Net-(U1-PB7_XTAL2)
- C3 pad 1: (no net) -> Net-(C3-Pad1)
- C3 pad 2: (no net) -> Net-(J2-Pin_2)
- C4 pad 1: (no net) -> Net-(C4-Pad1)
- C4 pad 2: (no net) -> Net-(J4-Pin_2)
- C5 pad 1: (no net) -> Net-(C5-Pad1)
- C5 pad 2: (no net) -> Net-(J5-Pin_2)
- Q1 pad 3: (no net) -> Net-(Q1-G)
- Q2 pad 1: (no net) -> Net-(Q2-B)
- R1 pad 1: (no net) -> Net-(U1-PC6_RESET)
- R12 pad 2: (no net) -> Net-(R12-Pad2)
- R14 pad 1: (no net) -> Net-(R14-Pad1)
- R2 pad 2: (no net) -> Net-(R2-Pad2)
- R24 pad 1: (no net) -> Net-(R24-Pad1)
- R3 pad 2: (no net) -> Net-(R3-Pad2)
- R31 pad 2: (no net) -> Net-(R31-Pad2)
- R4 pad 1: (no net) -> Net-(R4-Pad1)
- R5 pad 1: (no net) -> Net-(R5-Pad1)
- U1 pad 2: (no net) -> unconnected-(U1-PD0_RXD-Pad2)
- U1 pad 3: (no net) -> unconnected-(U1-PD1_TXD-Pad3)
- U13 pad 4: (no net) -> unconnected-(U13-RX-Pad4)
- U13 pad 6: (no net) -> unconnected-(U13-RST-Pad6)
- U13 pad 7: (no net) -> unconnected-(U13-CH-Pad7)
- U13 pad 8: (no net) -> unconnected-(U13-TX-Pad8)
Routing:
- net ADC1: track 267.4 -> 272.7 mm
- net Net-(J4-Pin_2): track 32.6 -> 33.2 mm
