File: Proyectos_KiCad/Dispensador_Garrafones_V2.0/Inputs.kicad_sch (KiCad schematic)
At the start: 25 parts, among them J11 FICHERO, Q6 2N3906, SW1 SW_DIP_x05, U11 PC817

Commit message: Nuevos Proyectos
Parts:
- C3, C4, C5: footprint Capacitor_THT:C_Disc_D3.8mm_W2.6mm_P2.50mm -> Capacitor_THT:C_Disc_D4.3mm_W1.9mm_P5.00mm
Changed lines of the file:
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@@
 			)
 		)
-		(property "Footprint" "Capacitor_THT:C_Disc_D3.8mm_W2.6mm_P2.50mm"
+		(property "Footprint" "Capacitor_THT:C_Disc_D4.3mm_W1.9mm_P5.00mm"
 			(at 191.77 50.8 0)
 			(effects
@@
 			)
 		)
-		(property "Footprint" "Capacitor_THT:C_Disc_D3.8mm_W2.6mm_P2.50mm"
+		(property "Footprint" "Capacitor_THT:C_Disc_D4.3mm_W1.9mm_P5.00mm"
 			(at 158.75 50.8 0)
 			(effects
@@
 			)
 		)
-		(property "Footprint" "Capacitor_THT:C_Disc_D3.8mm_W2.6mm_P2.50mm"
+		(property "Footprint" "Capacitor_THT:C_Disc_D4.3mm_W1.9mm_P5.00mm"
 			(at 124.46 50.8 0)
 			(effects

Commit message: Omarchy-RIP
Parts:
- J2, J3, J4: value ~ -> (none)
