File: Proyectos_KiCad/Dispensador_Garrafones_V2.0/Inputs.kicad_sch (KiCad schematic)
At the start: 25 parts, among them J11 FICHERO, Q6 2N3906, SW1 SW_DIP_x05, U11 PC817

Commit message: Backup antes de reinstalacion del SO: proyectos y librerias KiCad
Parts:
- renumbered C3 to C7, C4 to C8, C5 to C9, D9 to D7, J3 to J10, J11 to J7, J2 to J8, J4 to J9, R26 to R18, R4 to R19, R5 to R20, R6 to R21, R7 to R22, R8 to R23, R28 to R24, R27 to R25, R29 to R26, R2 to R27, R14 to R28, R3 to R29, SW1 to SW2, U11 to U8
