File: Proyectos_KiCad/Dispensador_Garrafones_V2.0/Microcontrolador.kicad_sch (KiCad schematic)
At the start: 7 parts, among them SW2 Push_Button, U8 Atmega328P-PU, Y1 Crystal_16MHz

Commit message: Nuevos Proyectos
Connections:
- net RELE_1: now also U8.11 (T1_PD5); no longer U8.4 (INT0_PD2)
- net RELE_2: now also U8.6 (T0_PD4); no longer U8.5 (INT1_PD3)
- net RELE_3: now also U8.5 (INT1_PD3); no longer U8.6 (T0_PD4)
- net RELE_4: now also U8.4 (INT0_PD2); no longer U8.11 (T1_PD5)
Changed lines of the file:
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@@
 		)
 	)
-	(hierarchical_label "RELE_4"
+	(hierarchical_label "RELE_1"
 		(shape input)
 		(at 142.24 77.47 0)
@@
 		)
 	)
-	(hierarchical_label "RELE_2"
+	(hierarchical_label "RELE_3"
 		(shape input)
 		(at 142.24 72.39 0)
@@
 		)
 	)
-	(hierarchical_label "RELE_1"
+	(hierarchical_label "RELE_4"
 		(shape input)
 		(at 142.24 69.85 0)
@@
 		)
 	)
-	(hierarchical_label "RELE_3"
+	(hierarchical_label "RELE_2"
 		(shape input)
 		(at 142.24 74.93 0)

Commit message: Omarchy-RIP
Parts:
- U10: value ~ -> (none)
