File: Proyectos_KiCad/Dispensador_Garrafones_V2.0/Microcontrolador.kicad_sch (KiCad schematic)
At the start: 7 parts, among them SW2 Push_Button, U8 Atmega328P-PU, Y1 Crystal_16MHz

Commit message: Backup antes de reinstalacion del SO: proyectos y librerias KiCad
Parts:
- renumbered C10 to C1, C11 to C2, R34 to R1, SW2 to SW1, U8 to U1, U10 to U2
Changed lines of the file:
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@@
 		(dnp no)
 		(fields_autoplaced yes)
-		(property "Reference" "#PWR07"
+		(property "Reference" "#PWR08"
 			(at 168.91 63.5 0)
 			(hide yes)
@@
 			(project "Dispensador_Garrafones_V2.0"
 				(path "/0292ef25-dc7e-42f1-b019-d6970f298ed7/92b91cc5-0e32-4296-854e-0c86d9840eee"
-					(reference "#PWR07")
+					(reference "#PWR08")
 					(unit 1)
 				)
@@
 		(dnp no)
 		(fields_autoplaced yes)
-		(property "Reference" "R34"
+		(property "Reference" "R1"
 			(at 99.06 44.4499 90)
 			(show_name no)
@@
 			(project "Dispensador_Garrafones_V2.0"
 				(path "/0292ef25-dc7e-42f1-b019-d6970f298ed7/92b91cc5-0e32-4296-854e-0c86d9840eee"
-					(reference "R34")
+					(reference "R1")
 					(unit 1)
 				)
@@
 		(dnp no)
 		(fields_autoplaced yes)
-		(property "Reference" "#PWR029"
+		(property "Reference" "#PWR01"
 			(at 68.58 88.9 0)
 			(hide yes)
@@
 			(project "Dispensador_Garrafones_V2.0"
 				(path "/0292ef25-dc7e-42f1-b019-d6970f298ed7/92b91cc5-0e32-4296-854e-0c86d9840eee"
-					(reference "#PWR029")
+					(reference "#PWR01")
 					(unit 1)
 				)
@@
 		(dnp no)
 		(fields_autoplaced yes)
-		(property "Reference" "U10"
+		(property "Reference" "U2"
 			(at 176.53 50.7999 0)
 			(show_name no)
@@
 			(project "Dispensador_Garrafones_V2.0"
 				(path "/0292ef25-dc7e-42f1-b019-d6970f298ed7/92b91cc5-0e32-4296-854e-0c86d9840eee"
-					(reference "U10")
+					(reference "U2")
 					(unit 1)
 				)
@@
 		(dnp no)
 		(fields_autoplaced yes)
-		(property "Reference" "#PWR06"
+		(property "Reference" "#PWR07"
 			(at 166.37 67.31 0)
 			(hide yes)
@@
 			(project "Dispensador_Garrafones_V2.0"
 				(path "/0292ef25-dc7e-42f1-b019-d6970f298ed7/92b91cc5-0e32-4296-854e-0c86d9840eee"
-					(reference "#PWR06")
+					(reference "#PWR07")
 					(unit 1)
 				)
@@
 		(dnp no)
 		(fields_autoplaced yes)
-		(property "Reference" "#PWR032"
+		(property "Reference" "#PWR06"
 			(at 91.44 97.79 0)
 			(hide yes)
@@
 			(project "Dispensador_Garrafones_V2.0"
 				(path "/0292ef25-dc7e-42f1-b019-d6970f298ed7/92b91cc5-0e32-4296-854e-0c86d9840eee"
-					(reference "#PWR032")
+					(reference "#PWR06")
 					(unit 1)
 				)
@@
 		(dnp no)
 		(fields_autoplaced yes)
-		(property "Reference" "C11"
+		(property "Reference" "C2"
 			(at 83.82 77.4762 0)
 			(show_name no)
@@
 			(project "Dispensador_Garrafones_V2.0"
 				(path "/0292ef25-dc7e-42f1-b019-d6970f298ed7/92b91cc5-0e32-4296-854e-0c86d9840eee"
-					(reference "C11")
+					(reference "C2")
 					(unit 1)
 				)
@@
 		(dnp no)
 		(fields_autoplaced yes)
-		(property "Reference" "SW2"
+		(property "Reference" "SW1"
 			(at 87.63 45.72 0)
 			(show_name no)
@@
 			(project "Dispensador_Garrafones_V2.0"
 				(path "/0292ef25-dc7e-42f1-b019-d6970f298ed7/92b91cc5-0e32-4296-854e-0c86d9840eee"
-					(reference "SW2")
+					(reference "SW1")
 					(unit 1)
 				)
@@
 		(dnp no)
 		(fields_autoplaced yes)
-		(property "Reference" "#PWR030"
+		(property "Reference" "#PWR03"
 			(at 81.28 88.9 0)
 			(hide yes)
@@
 			(project "Dispensador_Garrafones_V2.0"
 				(path "/0292ef25-dc7e-42f1-b019-d6970f298ed7/92b91cc5-0e32-4296-854e-0c86d9840eee"
-					(reference "#PWR030")
+					(reference "#PWR03")
 					(unit 1)
 				)
@@
 		(dnp no)
 		(fields_autoplaced yes)
-		(property "Reference" "#PWR031"
+		(property "Reference" "#PWR05"
 			(at 100.33 83.82 0)
 			(hide yes)
@@
 			(project "Dispensador_Garrafones_V2.0"
 				(path "/0292ef25-dc7e-42f1-b019-d6970f298ed7/92b91cc5-0e32-4296-854e-0c86d9840eee"
-					(reference "#PWR031")
+					(reference "#PWR05")
 					(unit 1)
 				)
@@
 		(dnp no)
 		(fields_autoplaced yes)
-		(property "Reference" "#PWR025"
+		(property "Reference" "#PWR02"
 			(at 73.66 53.34 0)
 			(hide yes)
@@
 			(project "Dispensador_Garrafones_V2.0"
 				(path "/0292ef25-dc7e-42f1-b019-d6970f298ed7/92b91cc5-0e32-4296-854e-0c86d9840eee"
-					(reference "#PWR025")
+					(reference "#PWR02")
 					(unit 1)
 				)
@@
 		(dnp no)
 		(fields_autoplaced yes)
-		(property "Reference" "#PWR026"
+		(property "Reference" "#PWR04"
 			(at 96.52 44.45 0)
 			(hide yes)
@@
 			(project "Dispensador_Garrafones_V2.0"
 				(path "/0292ef25-dc7e-42f1-b019-d6970f298ed7/92b91cc5-0e32-4296-854e-0c86d9840eee"
-					(reference "#PWR026")
+					(reference "#PWR04")
 					(unit 1)
 				)
@@
 		(dnp no)
 		(fields_autoplaced yes)
-		(property "Reference" "U8"
+		(property "Reference" "U1"
 			(at 120.65 45.72 0)
 			(show_name no)
@@
 			(project "Dispensador_Garrafones_V2.0"
 				(path "/0292ef25-dc7e-42f1-b019-d6970f298ed7/92b91cc5-0e32-4296-854e-0c86d9840eee"
-					(reference "U8")
+					(reference "U1")
 					(unit 1)
 				)
@@
 		(dnp no)
 		(fields_autoplaced yes)
-		(property "Reference" "C10"
+		(property "Reference" "C1"
 			(at 71.12 77.4762 0)
 			(show_name no)
@@
 			(project "Dispensador_Garrafones_V2.0"
 				(path "/0292ef25-dc7e-42f1-b019-d6970f298ed7/92b91cc5-0e32-4296-854e-0c86d9840eee"
-					(reference "C10")
-					(unit 1)
-				)
+					(reference "C1")
+					(unit 1)
+				)
