File: Proyectos_KiCad/Dispensador_Garrafones_V2.0/Outpus.kicad_sch (KiCad schematic)
At the start: 42 parts, among them J10 LOAD, J5 LOAD, J6 LOAD, J7 LOAD, J8 LOAD, J9 LOAD, Q1 TIP122, Q2 BT136-800, Q3 BT136-800, Q4 BT136-800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

Commit message: Nuevos Proyectos
Parts:
- Q1, Q2, Q3, Q4, Q5: footprint Package_TO_SOT_THT:TO-220-3_Vertical -> @EmersonPrez15:TO-220-3_VDC
- R15, R18, R22, R23: footprint PCM_Resistor_THT_AKL:R_Axial_DIN0207_L6.3mm_D2.5mm_P15.24mm_Horizontal -> Resistor_THT:R_Axial_DIN0207_L6.3mm_D2.5mm_P10.16mm_Horizontal
Connections:
- net ADC1: now also J10.1 (Pin_1); no longer J10.2 (Pin_2)
- net ADC2: now also J10.2 (Pin_2); no longer J10.1 (Pin_1)
- net VCC renamed +12V
Other:
- moved on the sheet: J5

Commit message: Omarchy-RIP
Parts:
- C6, C7, C8, C9: value C -> 10nF/400V
- D3, D5, D6, D7, D8: value ~ -> (none)
