File: Proyectos_KiCad/Dispensador_Garrafones_V2.0/Outpus.kicad_sch (KiCad schematic)
At the start: 42 parts, among them J10 LOAD, J5 LOAD, J6 LOAD, J7 LOAD, J8 LOAD, J9 LOAD, Q1 TIP122, Q2 BT136-800, Q3 BT136-800, Q4 BT136-800, Q5 BT136-800, U3 PC817, U4 MOC3021M, U5 MOC3021M, U6 MOC3021M, U7 MOC3021M

Commit message: Modificaciones GarrV2
Parts:
- added Q7: BTA41-600B, PCM_Package_TO_SOT_THT_AKL:TO-218-3_Vertical_AAG, symbol PCM_Triac_AKL:BTA41-600B
- J10, J6, J7, J8, J9: footprint TerminalBlock_Phoenix:TerminalBlock_Phoenix_MKDS-1,5-2-5.08_1x02_P5.08mm_Horizontal -> Connector_AMASS:AMASS_XT30U-F_1x02_P5.0mm_Vertical
- Q2, Q3, Q4, Q5: footprint @EmersonPrez15:TO-220-3_VDC -> PCM_Package_TO_SOT_THT_AKL:TO-3P-3_Vertical
Changed lines of the file:
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@@
 			)
 		)
-		(property "Footprint" "@EmersonPrez15:TO-220-3_VDC"
+		(property "Footprint" "PCM_Package_TO_SOT_THT_AKL:TO-3P-3_Vertical"
 			(at 254 74.295 0)
 			(hide yes)
@@
 			)
 		)
-		(property "Footprint" "@EmersonPrez15:TO-220-3_VDC"
+		(property "Footprint" "PCM_Package_TO_SOT_THT_AKL:TO-3P-3_Vertical"
 			(at 254 38.735 0)
 			(hide yes)
@@
 			)
 		)
-		(property "Footprint" "@EmersonPrez15:TO-220-3_VDC"
+		(property "Footprint" "PCM_Package_TO_SOT_THT_AKL:TO-3P-3_Vertical"
 			(at 166.37 74.295 0)
 			(hide yes)
@@
 			)
 		)
-		(property "Footprint" "TerminalBlock_Phoenix:TerminalBlock_Phoenix_MKDS-1,5-2-5.08_1x02_P5.08mm_Horizontal"
+		(property "Footprint" "Connector_AMASS:AMASS_XT30U-F_1x02_P5.0mm_Vertical"
 			(at 130.81 95.25 0)
 			(hide yes)
@@
 			)
 		)
-		(property "Footprint" "TerminalBlock_Phoenix:TerminalBlock_Phoenix_MKDS-1,5-2-5.08_1x02_P5.08mm_Horizontal"
+		(property "Footprint" "Connector_AMASS:AMASS_XT30U-F_1x02_P5.0mm_Vertical"
 			(at 273.05 76.2 0)
 			(hide yes)
@@
 			)
 		)
-		(property "Footprint" "@EmersonPrez15:TO-220-3_VDC"
+		(property "Footprint" "PCM_Package_TO_SOT_THT_AKL:TO-3P-3_Vertical"
 			(at 166.37 38.735 0)
 			(hide yes)
@@
 			)
 		)
-		(property "Footprint" "TerminalBlock_Phoenix:TerminalBlock_Phoenix_MKDS-1,5-2-5.08_1x02_P5.08mm_Horizontal"
+		(property "Footprint" "Connector_AMASS:AMASS_XT30U-F_1x02_P5.0mm_Vertical"
 			(at 185.42 40.64 0)
 			(hide yes)
@@
 			)
 		)
-		(property "Footprint" "TerminalBlock_Phoenix:TerminalBlock_Phoenix_MKDS-1,5-2-5.08_1x02_P5.08mm_Horizontal"
+		(property "Footprint" "Connector_AMASS:AMASS_XT30U-F_1x02_P5.0mm_Vertical"
 			(at 185.42 76.2 0)
 			(hide yes)
@@
 	)
 	(symbol
+		(lib_id "PCM_Triac_AKL:BTA41-600B")
+		(at 162.56 91.44 0)
+		(unit 1)
+		(body_style 1)
+		(exclude_from_sim no)
+		(in_bom yes)
+		(on_board yes)
+		(in_pos_files yes)
+		(dnp no)
+		(fields_autoplaced yes)
+		(property "Reference" "Q7"
+			(at 166.37 90.1699 0)
+			(show_name no)
+			(do_not_autoplace no)
+			(effects
+				(font
+					(size 1.27 1.27)
+				)
+				(justify left)
+			)
+		)
+		(property "Value" "BTA41-600B"
+			(at 166.37 92.7099 0)
+			(show_name no)
+			(do_not_autoplace no)
+			(effects
+				(font
+					(size 1.27 1.27)
+				)
+				(justify left)
+			)
+		)
+		(property "Footprint" "PCM_Package_TO_SOT_THT_AKL:TO-218-3_Vertical_AAG"
+			(at 162.56 91.44 0)
+			(hide yes)
+			(show_name no)
+			(do_not_autoplace no)
+			(effects
+				(font
+					(size 1.27 1.27)
+				)
+			)
+		)
+		(property "Datasheet" "https://www.tme.eu/Document/04a7384ba2314a2a2c0be567aaa7f9a3/BTA41-800BRG-STMicroelectronics.pdf"
+			(at 162.56 91.44 0)
+			(hide yes)
+			(show_name no)
+			(do_not_autoplace no)
+			(effects
+				(font
+					(size 1.27 1.27)
+				)
+			)
+		)
+		(property "Description" "TO-218 Triac, 600V, 41A, Alternate KiCAD Library"
+			(at 162.56 91.44 0)
+			(hide yes)
+			(show_name no)
+			(do_not_autoplace no)
+			(effects
+				(font
+					(size 1.27 1.27)
+				)
+			)
+		)
+		(pin "2"
+		)
+		(pin "1"
+		)
+		(pin "3"
+		)
+		(instances
+			(project "Dispensador_Garrafones_V2.0"
+				(path "/0292ef25-dc7e-42f1-b019-d6970f298ed7/e2024343-7001-4b21-9393-3bf97457ac68"
+					(reference "Q7")
+					(unit 1)
+				)
+			)
+		)
+	)
+	(symbol
 		(lib_id "Device:R_Small")
 		(at 60.96 59.69 90)
@@
 			)
 		)
-		(property "Footprint" "TerminalBlock_Phoenix:TerminalBlock_Phoenix_MKDS-1,5-2-5.08_1x02_P5.08mm_Horizontal"
+		(property "Footprint" "Connector_AMASS:AMASS_XT30U-F_1x02_P5.0mm_Vertical"
 			(at 273.05 40.64 0)
 			(hide yes)

Commit message: Backup antes de reinstalacion del SO: proyectos y librerias KiCad
Parts:
- removed Q7: BTA41-600B, PCM_Package_TO_SOT_THT_AKL:TO-218-3_Vertical_AAG, symbol PCM_Triac_AKL:BTA41-600B
- renumbered C6 to C3, C7 to C4, C8 to C5, C9 to C6, D5 to D1, D3 to D2, D4 to D3, D6 to D4, D7 to D5, D8 to D6, J10 to J1, J7 to J2, J5 to J3, J8 to J4, J6 to J5, J9 to J6, Q2 to Q1, Q1 to Q2, R18 to R10, R19 to R11, R17 to R12, R21 to R13, R22 to R14, R23 to R15, R24 to R16, R25 to R17, R9 to R2, R13 to R3, R10 to R4, R15 to R5, R11 to R6, R12 to R7, R16 to R8, R20 to R9, U6 to U5, U5 to U6
Other:
- moved on the sheet: C3, C4, D1, D4, J1, J2, J4, Q1, Q3, R10, R11, R3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
