File: Proyectos_KiCad/Dispensador_Garrafones_V2.0/Power.kicad_sch (KiCad schematic)
At the start: 12 parts, among them J1 JACK_DC, U1 MP1584, U2 AMS1117-3.3

Commit message: Modificaciones GarrV2
Connections:
- net +12V: now also U1.2 (IN-); no longer U1.1 (IN+)
- net GND: now also U1.1 (IN+), U1.3 (+OUT); no longer U1.2 (IN-), U1.4 (-OUT)
- net at D1.2 (A): now also U1.4 (-OUT); no longer U1.3 (+OUT)
Changed lines of the file:
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@@
+	(wire
+		(pts
+			(xy 73.66 45.72) (xy 77.47 45.72)
+		)
+		(stroke
+			(width 0)
+			(type default)
+		)
+	)
 	(wire
 		(pts
@@
 	(wire
 		(pts
+			(xy 123.19 45.72) (xy 123.19 49.53)
+		)
+		(stroke
+			(width 0)
+			(type default)
+		)
+	)
+	(wire
+		(pts
+			(xy 105.41 41.91) (xy 105.41 45.72)
+		)
+		(stroke
+			(width 0)
+			(type default)
+		)
+	)
+	(wire
+		(pts
+			(xy 105.41 45.72) (xy 104.14 45.72)
+		)
+		(stroke
+			(width 0)
+			(type default)
+		)
+	)
+	(wire
+		(pts
+			(xy 69.85 59.69) (xy 69.85 50.8)
+		)
+		(stroke
+			(width 0)
+			(type default)
+		)
+	)
+	(wire
+		(pts
+			(xy 73.66 43.18) (xy 73.66 45.72)
+		)
+		(stroke
+			(width 0)
+			(type default)
+		)
+	)
+	(wire
+		(pts
+			(xy 146.05 45.72) (xy 146.05 49.53)
+		)
+		(stroke
+			(width 0)
+			(type default)
+		)
+	)
+	(wire
+		(pts
+			(xy 111.76 41.91) (xy 111.76 44.45)
+		)
+		(stroke
+			(width 0)
+			(type default)
+		)
+	)
+	(wire
+		(pts
+			(xy 69.85 48.26) (xy 69.85 50.8)
+		)
+		(stroke
+			(width 0)
+			(type default)
+		)
+	)
+	(wire
+		(pts
+			(xy 74.93 59.69) (xy 74.93 50.8)
+		)
+		(stroke
+			(width 0)
+			(type default)
+		)
+	)
+	(wire
+		(pts
+			(xy 146.05 45.72) (xy 146.05 43.18)
+		)
+		(stroke
+			(width 0)
+			(type default)
+		)
+	)
+	(wire
+		(pts
+			(xy 97.79 50.8) (xy 97.79 59.69)
+		)
+		(stroke
+			(width 0)
+			(type default)
+		)
+	)
+	(wire
+		(pts
+			(xy 123.19 41.91) (xy 123.19 45.72)
+		)
+		(stroke
+			(width 0)
+			(type default)
+		)
+	)
+	(wire
+		(pts
+			(xy 111.76 57.15) (xy 111.76 59.69)
+		)
+		(stroke
+			(width 0)
+			(type default)
+		)
+	)
+	(wire
+		(pts
+			(xy 146.05 54.61) (xy 146.05 59.69)
+		)
+		(stroke
+			(width 0)
+			(type default)
+		)
+	)
+	(wire
+		(pts
+			(xy 67.31 48.26) (xy 69.85 48.26)
+		)
+		(stroke
+			(width 0)
+			(type default)
+		)
+	)
+	(wire
+		(pts
+			(xy 74.93 50.8) (xy 77.47 50.8)
+		)
+		(stroke
+			(width 0)
+			(type default)
+		)
+	)
+	(wire
+		(pts
 			(xy 95.25 50.8) (xy 97.79 50.8)
 		)
@@
 	(wire
 		(pts
-			(xy 123.19 45.72) (xy 123.19 49.53)
-		)
-		(stroke
-			(width 0)
-			(type default)
-		)
-	)
-	(wire
-		(pts
-			(xy 105.41 41.91) (xy 105.41 45.72)
-		)
-		(stroke
-			(width 0)
-			(type default)
-		)
-	)
-	(wire
-		(pts
-			(xy 105.41 45.72) (xy 104.14 45.72)
-		)
-		(stroke
-			(width 0)
-			(type default)
-		)
-	)
-	(wire
-		(pts
-			(xy 69.85 59.69) (xy 69.85 50.8)
-		)
-		(stroke
-			(width 0)
-			(type default)
-		)
-	)
-	(wire
-		(pts
-			(xy 73.66 43.18) (xy 73.66 45.72)
-		)
-		(stroke
-			(width 0)
-			(type default)
-		)
-	)
-	(wire
-		(pts
-			(xy 146.05 45.72) (xy 146.05 49.53)
-		)
-		(stroke
-			(width 0)
-			(type default)
-		)
-	)
-	(wire
-		(pts
-			(xy 111.76 41.91) (xy 111.76 44.45)
-		)
-		(stroke
-			(width 0)
-			(type default)
-		)
-	)
-	(wire
-		(pts
-			(xy 69.85 48.26) (xy 69.85 50.8)
-		)
-		(stroke
-			(width 0)
-			(type default)
-		)
-	)
-	(wire
-		(pts
-			(xy 74.93 59.69) (xy 74.93 50.8)
-		)
-		(stroke
-			(width 0)
-			(type default)
-		)
-	)
-	(wire
-		(pts
-			(xy 146.05 45.72) (xy 146.05 43.18)
-		)
-		(stroke
-			(width 0)
-			(type default)
-		)
-	)
-	(wire
-		(pts
-			(xy 97.79 50.8) (xy 97.79 59.69)
-		)
-		(stroke
-			(width 0)
-			(type default)
-		)
-	)
-	(wire
-		(pts
-			(xy 123.19 41.91) (xy 123.19 45.72)
-		)
-		(stroke
-			(width 0)
-			(type default)
-		)
-	)
-	(wire
-		(pts
-			(xy 111.76 57.15) (xy 111.76 59.69)
-		)
-		(stroke
-			(width 0)
-			(type default)
-		)
-	)
-	(wire
-		(pts
-			(xy 146.05 54.61) (xy 146.05 59.69)
-		)
-		(stroke
-			(width 0)
-			(type default)
-		)
-	)
-	(wire
-		(pts
-			(xy 67.31 48.26) (xy 69.85 48.26)
-		)
-		(stroke
-			(width 0)
-			(type default)
-		)
-	)
-	(wire
-		(pts
 			(xy 67.31 45.72) (xy 73.66 45.72)
 		)
@@
 		(pts
 			(xy 123.19 45.72) (xy 127 45.72)
-		)
-		(stroke
-			(width 0)
-			(type default)
-		)
-	)
-	(wire
-		(pts
-			(xy 73.66 45.72) (xy 77.47 45.72)
-		)
-		(stroke
-			(width 0)
-			(type default)
-		)
-	)
-	(wire
-		(pts
-			(xy 74.93 50.8) (xy 77.47 50.8)
 		)
 		(stroke
@@
 		(lib_id "@EmersonPrez15:MP1584")
 		(at 86.36 48.26 0)
+		(mirror x)
 		(unit 1)
 		(body_style 1)
@@
 		(in_pos_files yes)
 		(dnp no)
-		(fields_autoplaced yes)
 		(property "Reference" "U1"
-			(at 86.36 39.37 0)
+			(at 86.36 57.15 0)
 			(show_name no)
 			(do_not_autoplace no)
@@
 		)
 		(property "Value" "MP1584"
-			(at 86.36 41.91 0)
-			(show_name no)
-			(do_not_autoplace no)
+			(at 86.36 54.61 0)
+			(show_name no)
+			(do_not_autoplace no)

Commit message: Backup antes de reinstalacion del SO: proyectos y librerias KiCad
Parts:
- renumbered C1 to C10, C2 to C11, D1 to D8, D2 to D9, J1 to J11, R1 to R30, U2 to U10, U1 to U9
Changed lines of the file:
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@@
 		(dnp no)
 		(fields_autoplaced yes)
-		(property "Reference" "#PWR0114"
+		(property "Reference" "#PWR039"
 			(at 74.93 66.04 0)
 			(hide yes)
@@
 			(project "Dispensador_Garrafones_V2.0"
 				(path "/0292ef25-dc7e-42f1-b019-d6970f298ed7/0f400d35-56c5-49e0-b18b-32396a436e4b"
-					(reference "#PWR0114")
+					(reference "#PWR039")
 					(unit 1)
 				)
@@
 		(in_pos_files yes)
 		(dnp no)
-		(property "Reference" "D2"
+		(property "Reference" "D9"
 			(at 114.3 53.9114 90)
 			(show_name no)
@@
 			(project "Dispensador_Garrafones_V2.0"
 				(path "/0292ef25-dc7e-42f1-b019-d6970f298ed7/0f400d35-56c5-49e0-b18b-32396a436e4b"
-					(reference "D2")
+					(reference "D9")
 					(unit 1)
 				)
@@
 		(dnp no)
 		(fields_autoplaced yes)
-		(property "Reference" "#PWR0115"
+		(property "Reference" "#PWR037"
 			(at 69.85 66.04 0)
 			(hide yes)
@@
 			(project "Dispensador_Garrafones_V2.0"
 				(path "/0292ef25-dc7e-42f1-b019-d6970f298ed7/0f400d35-56c5-49e0-b18b-32396a436e4b"
-					(reference "#PWR0115")
+					(reference "#PWR037")
 					(unit 1)
 				)
@@
 		(dnp no)
 		(fields_autoplaced yes)
-		(property "Reference" "#PWR0118"
+		(property "Reference" "#PWR043"
 			(at 111.76 66.04 0)
 			(hide yes)
@@
 			(project "Dispensador_Garrafones_V2.0"
 				(path "/0292ef25-dc7e-42f1-b019-d6970f298ed7/0f400d35-56c5-49e0-b18b-32396a436e4b"
-					(reference "#PWR0118")
+					(reference "#PWR043")
 					(unit 1)
 				)
@@
 		(in_pos_files yes)
 		(dnp no)
-		(property "Reference" "C2"
+		(property "Reference" "C11"
 			(at 148.59 50.2538 0)
 			(show_name no)
@@
 			(project "Dispensador_Garrafones_V2.0"
 				(path "/0292ef25-dc7e-42f1-b019-d6970f298ed7/0f400d35-56c5-49e0-b18b-32396a436e4b"
-					(reference "C2")
+					(reference "C11")
 					(unit 1)
 				)
@@
 		(dnp no)
 		(fields_autoplaced yes)
-		(property "Reference" "#PWR0112"
+		(property "Reference" "#PWR041"
 			(at 105.41 45.72 0)
 			(hide yes)
@@
 			(project "Dispensador_Garrafones_V2.0"
 				(path "/0292ef25-dc7e-42f1-b019-d6970f298ed7/0f400d35-56c5-49e0-b18b-32396a436e4b"
-					(reference "#PWR0112")
+					(reference "#PWR041")
 					(unit 1)
 				)
@@
 		(in_pos_files yes)
 		(dnp no)
-		(property "Reference" "R1"
+		(property "Reference" "R30"
 			(at 114.3 45.7199 0)
 			(hide yes)
@@
 			(project "Dispensador_Garrafones_V2.0"
 				(path "/0292ef25-dc7e-42f1-b019-d6970f298ed7/0f400d35-56c5-49e0-b18b-32396a436e4b"
-					(reference "R1")
+					(reference "R30")
 					(unit 1)
 				)
@@
 		(dnp no)
 		(fields_autoplaced yes)
-		(property "Reference" "#PWR0123"
+		(property "Reference" "#PWR048"
 			(at 146.05 66.04 0)
 			(hide yes)
@@
 			(project "Dispensador_Garrafones_V2.0"
 				(path "/0292ef25-dc7e-42f1-b019-d6970f298ed7/0f400d35-56c5-49e0-b18b-32396a436e4b"
-					(reference "#PWR0123")
+					(reference "#PWR048")
 					(unit 1)
 				)
@@
 		(in_pos_files yes)
 		(dnp no)
-		(property "Reference" "U1"
+		(property "Reference" "U9"
 			(at 86.36 57.15 0)
 			(show_name no)
@@
 			(project "Dispensador_Garrafones_V2.0"
 				(path "/0292ef25-dc7e-42f1-b019-d6970f298ed7/0f400d35-56c5-49e0-b18b-32396a436e4b"
-					(reference "U1")
+					(reference "U9")
 					(unit 1)
 				)
@@
 		(dnp no)
 		(fields_autoplaced yes)
-		(property "Reference" "U2"
+		(property "Reference" "U10"
 			(at 134.62 39.37 0)
 			(show_name no)
@@
 			(project "Dispensador_Garrafones_V2.0"
 				(path "/0292ef25-dc7e-42f1-b019-d6970f298ed7/0f400d35-56c5-49e0-b18b-32396a436e4b"
-					(reference "U2")
+					(reference "U10")
 					(unit 1)
 				)
@@
 		(dnp no)
 		(fields_autoplaced yes)
-		(property "Reference" "#PWR036"
+		(property "Reference" "#PWR038"
 			(at 73.66 46.99 0)
 			(hide yes)
@@
 			(project "Dispensador_Garrafones_V2.0"
 				(path "/0292ef25-dc7e-42f1-b019-d6970f298ed7/0f400d35-56c5-49e0-b18b-32396a436e4b"
-					(reference "#PWR036")
+					(reference "#PWR038")
 					(unit 1)
 				)
@@
 		(dnp no)
 		(fields_autoplaced yes)
-		(property "Reference" "#PWR0119"
+		(property "Reference" "#PWR042"
 			(at 111.76 45.72 0)
 			(hide yes)
@@
 			(project "Dispensador_Garrafones_V2.0"
 				(path "/0292ef25-dc7e-42f1-b019-d6970f298ed7/0f400d35-56c5-49e0-b18b-32396a436e4b"
-					(reference "#PWR0119")
+					(reference "#PWR042")
 					(unit 1)
 				)
@@
 		(dnp no)
 		(fields_autoplaced yes)
-		(property "Reference" "#PWR0113"
+		(property "Reference" "#PWR040"
 			(at 97.79 66.04 0)
 			(hide yes)
@@
 			(project "Dispensador_Garrafones_V2.0"
 				(path "/0292ef25-dc7e-42f1-b019-d6970f298ed7/0f400d35-56c5-49e0-b18b-32396a436e4b"
-					(reference "#PWR0113")
+					(reference "#PWR040")
 					(unit 1)
 				)
@@
 		(dnp no)
 		(fields_autoplaced yes)
-		(property "Reference" "#PWR0120"
+		(property "Reference" "#PWR044"
 			(at 123.19 45.72 0)
 			(hide yes)
@@
 			(project "Dispensador_Garrafones_V2.0"
 				(path "/0292ef25-dc7e-42f1-b019-d6970f298ed7/0f400d35-56c5-49e0-b18b-32396a436e4b"
-					(reference "#PWR0120")
+					(reference "#PWR044")
 					(unit 1)
 				)
@@
 		(in_pos_files yes)
 		(dnp no)
-		(property "Reference" "C1"
+		(property "Reference" "C10"
 			(at 125.73 50.2538 0)
 			(show_name no)
@@
 			(project "Dispensador_Garrafones_V2.0"
 				(path "/0292ef25-dc7e-42f1-b019-d6970f298ed7/0f400d35-56c5-49e0-b18b-32396a436e4b"
-					(reference "C1")
+					(reference "C10")
 					(unit 1)
 				)
@@
 		(dnp no)
 		(fields_autoplaced yes)
-		(property "Reference" "#PWR0117"
+		(property "Reference" "#PWR045"
 			(at 123.19 66.04 0)
 			(hide yes)
@@
 			(project "Dispensador_Garrafones_V2.0"
 				(path "/0292ef25-dc7e-42f1-b019-d6970f298ed7/0f400d35-56c5-49e0-b18b-32396a436e4b"
-					(reference "#PWR0117")
+					(reference "#PWR045")
 					(unit 1)
 				)
@@
 		(dnp no)
 		(fields_autoplaced yes)
-		(property "Reference" "D1"
+		(property "Reference" "D8"
 			(at 100.33 39.37 0)
 			(show_name no)
@@
 			(project "Dispensador_Garrafones_V2.0"
 				(path "/0292ef25-dc7e-42f1-b019-d6970f298ed7/0f400d35-56c5-49e0-b18b-32396a436e4b"
-					(reference "D1")
+					(reference "D8")
 					(unit 1)
 				)
@@
 		(dnp no)
 		(fields_autoplaced yes)
-		(property "Reference" "#PWR0122"
+		(property "Reference" "#PWR046"
 			(at 134.62 66.04 0)
 			(hide yes)
@@
 			(project "Dispensador_Garrafones_V2.0"
 				(path "/0292ef25-dc7e-42f1-b019-d6970f298ed7/0f400d35-56c5-49e0-b18b-32396a436e4b"
-					(reference "#PWR0122")
+					(reference "#PWR046")
 					(unit 1)
 				)
@@
 		(in_pos_files yes)
 		(dnp no)
-		(property "Reference" "J1"
+		(property "Reference" "J11"
 			(at 59.69 39.37 0)
 			(show_name no)
@@
 			(project "Dispensador_Garrafones_V2.0"
 				(path "/0292ef25-dc7e-42f1-b019-d6970f298ed7/0f400d35-56c5-49e0-b18b-32396a436e4b"
-					(reference "J1")
+					(reference "J11")
 					(unit 1)
 				)
@@
 		(dnp no)
 		(fields_autoplaced yes)
-		(property "Reference" "#PWR0121"
+		(property "Reference" "#PWR047"
 			(at 146.05 46.99 0)
 			(hide yes)
@@
 			(project "Dispensador_Garrafones_V2.0"
 				(path "/0292ef25-dc7e-42f1-b019-d6970f298ed7/0f400d35-56c5-49e0-b18b-32396a436e4b"
-					(reference "#PWR0121")
-					(unit 1)
-				)
+					(reference "#PWR047")
+					(unit 1)
+				)
