File: Proyectos_KiCad/Dispensador_Garrafones_V2.0/ESP01.kicad_sch (KiCad schematic)
At the start: 7 parts, among them U12 PC817, U13 PC817, U9 ESP-01S

Commit message: Backup antes de reinstalacion del SO: proyectos y librerias KiCad
Parts:
- renumbered R30 to R31, R31 to R33, R33 to R34, U12 to U11, U13 to U12, U9 to U13
Changed lines of the file:
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@@
 		(dnp no)
 		(fields_autoplaced yes)
-		(property "Reference" "#PWR020"
+		(property "Reference" "#PWR052"
 			(at 160.02 53.34 0)
 			(hide yes)
@@
 			(project "Dispensador_Garrafones_V2.0"
 				(path "/0292ef25-dc7e-42f1-b019-d6970f298ed7/6e10854a-81d1-4cb3-a96c-d4aac551c98c"
-					(reference "#PWR020")
+					(reference "#PWR052")
 					(unit 1)
 				)
@@
 		(dnp no)
 		(fields_autoplaced yes)
-		(property "Reference" "U13"
+		(property "Reference" "U12"
 			(at 148.59 68.58 0)
 			(show_name no)
@@
 			(project "Dispensador_Garrafones_V2.0"
 				(path "/0292ef25-dc7e-42f1-b019-d6970f298ed7/6e10854a-81d1-4cb3-a96c-d4aac551c98c"
-					(reference "U13")
+					(reference "U12")
 					(unit 1)
 				)
@@
 		(dnp no)
 		(fields_autoplaced yes)
-		(property "Reference" "R30"
+		(property "Reference" "R31"
 			(at 134.62 33.02 0)
 			(show_name no)
@@
 			(project "Dispensador_Garrafones_V2.0"
 				(path "/0292ef25-dc7e-42f1-b019-d6970f298ed7/6e10854a-81d1-4cb3-a96c-d4aac551c98c"
-					(reference "R30")
+					(reference "R31")
 					(unit 1)
 				)
@@
 		(dnp no)
 		(fields_autoplaced yes)
-		(property "Reference" "U12"
+		(property "Reference" "U11"
 			(at 148.59 33.02 0)
 			(show_name no)
@@
 			(project "Dispensador_Garrafones_V2.0"
 				(path "/0292ef25-dc7e-42f1-b019-d6970f298ed7/6e10854a-81d1-4cb3-a96c-d4aac551c98c"
-					(reference "U12")
+					(reference "U11")
 					(unit 1)
 				)
@@
 		(dnp no)
 		(fields_autoplaced yes)
-		(property "Reference" "#PWR018"
+		(property "Reference" "#PWR056"
 			(at 217.17 53.34 0)
 			(hide yes)
@@
 			(project "Dispensador_Garrafones_V2.0"
 				(path "/0292ef25-dc7e-42f1-b019-d6970f298ed7/6e10854a-81d1-4cb3-a96c-d4aac551c98c"
-					(reference "#PWR018")
+					(reference "#PWR056")
 					(unit 1)
 				)
@@
 		(dnp no)
 		(fields_autoplaced yes)
-		(property "Reference" "#PWR019"
+		(property "Reference" "#PWR049"
 			(at 138.43 53.34 0)
 			(hide yes)
@@
 			(project "Dispensador_Garrafones_V2.0"
 				(path "/0292ef25-dc7e-42f1-b019-d6970f298ed7/6e10854a-81d1-4cb3-a96c-d4aac551c98c"
-					(reference "#PWR019")
+					(reference "#PWR049")
 					(unit 1)
 				)
@@
 		(dnp no)
 		(fields_autoplaced yes)
-		(property "Reference" "#PWR021"
+		(property "Reference" "#PWR051"
 			(at 160.02 30.48 0)
 			(hide yes)
@@
 			(project "Dispensador_Garrafones_V2.0"
 				(path "/0292ef25-dc7e-42f1-b019-d6970f298ed7/6e10854a-81d1-4cb3-a96c-d4aac551c98c"
-					(reference "#PWR021")
+					(reference "#PWR051")
 					(unit 1)
 				)
@@
 		(dnp no)
 		(fields_autoplaced yes)
-		(property "Reference" "#PWR017"
+		(property "Reference" "#PWR055"
 			(at 184.15 45.72 0)
 			(hide yes)
@@
 			(project "Dispensador_Garrafones_V2.0"
 				(path "/0292ef25-dc7e-42f1-b019-d6970f298ed7/6e10854a-81d1-4cb3-a96c-d4aac551c98c"
-					(reference "#PWR017")
+					(reference "#PWR055")
 					(unit 1)
 				)
@@
 		(dnp no)
 		(fields_autoplaced yes)
-		(property "Reference" "U9"
+		(property "Reference" "U13"
 			(at 207.01 38.1 0)
 			(show_name no)
@@
 			(project "Dispensador_Garrafones_V2.0"
 				(path "/0292ef25-dc7e-42f1-b019-d6970f298ed7/6e10854a-81d1-4cb3-a96c-d4aac551c98c"
-					(reference "U9")
+					(reference "U13")
 					(unit 1)
 				)
@@
 		(dnp no)
 		(fields_autoplaced yes)
-		(property "Reference" "R31"
+		(property "Reference" "R33"
 			(at 162.56 31.7499 90)
 			(show_name no)
@@
 			(project "Dispensador_Garrafones_V2.0"
 				(path "/0292ef25-dc7e-42f1-b019-d6970f298ed7/6e10854a-81d1-4cb3-a96c-d4aac551c98c"
-					(reference "R31")
+					(reference "R33")
 					(unit 1)
 				)
@@
 		(dnp no)
 		(fields_autoplaced yes)
-		(property "Reference" "#PWR024"
+		(property "Reference" "#PWR054"
 			(at 160.02 88.9 0)
 			(hide yes)
@@
 			(project "Dispensador_Garrafones_V2.0"
 				(path "/0292ef25-dc7e-42f1-b019-d6970f298ed7/6e10854a-81d1-4cb3-a96c-d4aac551c98c"
-					(reference "#PWR024")
+					(reference "#PWR054")
 					(unit 1)
 				)
@@
 		(dnp no)
 		(fields_autoplaced yes)
-		(property "Reference" "#PWR023"
+		(property "Reference" "#PWR053"
 			(at 160.02 66.04 0)
 			(hide yes)
@@
 			(project "Dispensador_Garrafones_V2.0"
 				(path "/0292ef25-dc7e-42f1-b019-d6970f298ed7/6e10854a-81d1-4cb3-a96c-d4aac551c98c"
-					(reference "#PWR023")
+					(reference "#PWR053")
 					(unit 1)
 				)
@@
 		(dnp no)
 		(fields_autoplaced yes)
-		(property "Reference" "#PWR022"
+		(property "Reference" "#PWR050"
 			(at 138.43 88.9 0)
 			(hide yes)
@@
 			(project "Dispensador_Garrafones_V2.0"
 				(path "/0292ef25-dc7e-42f1-b019-d6970f298ed7/6e10854a-81d1-4cb3-a96c-d4aac551c98c"
-					(reference "#PWR022")
+					(reference "#PWR050")
 					(unit 1)
 				)
@@
 		(dnp no)
 		(fields_autoplaced yes)
-		(property "Reference" "R33"
+		(property "Reference" "R34"
 			(at 162.56 67.3099 90)
 			(show_name no)
@@
 			(project "Dispensador_Garrafones_V2.0"
 				(path "/0292ef25-dc7e-42f1-b019-d6970f298ed7/6e10854a-81d1-4cb3-a96c-d4aac551c98c"
-					(reference "R33")
-					(unit 1)
-				)
+					(reference "R34")
+					(unit 1)
+				)
