File: Proyectos_KiCad/555_ASIN/555_ASIN.kicad_pcb (KiCad board)
At the start: 2 copper layers, 45 x 45 mm, 16 parts, among them J1 VINPUT, J2 SWITCH, J3 POT, J4 OUTPUT, Q1 TIP49, U1 555

Commit message: Backup antes de reinstalacion del SO: proyectos y librerias KiCad
Parts:
- D2: footprint PCM_Diode_THT_AKL:D_DO-41_SOD81_P7.62mm_Horizontal -> PCM_Diode_THT_AKL_local:D_DO-41_SOD81_P7.62mm_Horizontal
- Q1: footprint PCM_Package_TO_SOT_THT_AKL:TO-220-3_Vertical_BCE -> PCM_Package_TO_SOT_THT_AKL_local:TO-220-3_Vertical_BCE
- U1: footprint PCM_Package_DIP_AKL:DIP-8_W7.62mm_LongPads -> PCM_Package_DIP_AKL_local:DIP-8_W7.62mm_LongPads
