File: Proyectos_KiCad/555_ASIN/555_ASIN.kicad_sch (KiCad schematic)
At the start: 16 parts, among them J1 VINPUT, J2 SWITCH, J3 POT, J4 OUTPUT, Q1 TIP49, U1 555

Commit message: Backup antes de reinstalacion del SO: proyectos y librerias KiCad
Parts:
- D2: symbol PCM_Diode_AKL:1N4004 -> PCM_Diode_AKL_local:1N4004
- Q1: symbol PCM_Transistor_BJT_AKL:TIP49 -> PCM_Transistor_BJT_AKL_local:TIP49
Changed lines of the file:
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@@
 	)
 	(symbol
-		(lib_id "PCM_SparkFun-PowerSymbol:GND")
+		(lib_id "PCM_SparkFun-PowerSymbol_local:GND")
 		(at 161.29 67.31 0)
 		(unit 1)
@@
 	)
 	(symbol
-		(lib_id "PCM_SparkFun-PowerSymbol:VIN")
+		(lib_id "PCM_SparkFun-PowerSymbol_local:VIN")
 		(at 142.24 34.29 0)
 		(unit 1)
@@
 	)
 	(symbol
-		(lib_id "PCM_SparkFun-PowerSymbol:GND")
+		(lib_id "PCM_SparkFun-PowerSymbol_local:GND")
 		(at 142.24 67.31 0)
 		(unit 1)
@@
 	)
 	(symbol
-		(lib_id "PCM_SparkFun-PowerSymbol:VIN")
+		(lib_id "PCM_SparkFun-PowerSymbol_local:VIN")
 		(at 130.81 34.29 0)
 		(unit 1)
@@
 	)
 	(symbol
-		(lib_id "PCM_SparkFun-PowerSymbol:GND")
+		(lib_id "PCM_SparkFun-PowerSymbol_local:GND")
 		(at 177.8 67.31 0)
 		(unit 1)
@@
 	)
 	(symbol
-		(lib_id "PCM_SparkFun-PowerSymbol:GND")
+		(lib_id "PCM_SparkFun-PowerSymbol_local:GND")
 		(at 86.36 62.23 0)
 		(unit 1)
@@
 	)
 	(symbol
-		(lib_id "PCM_SparkFun-PowerSymbol:VIN")
+		(lib_id "PCM_SparkFun-PowerSymbol_local:VIN")
 		(at 114.3 40.64 0)
 		(unit 1)
@@
 	)
 	(symbol
-		(lib_id "PCM_SparkFun-PowerSymbol:VCC")
+		(lib_id "PCM_SparkFun-PowerSymbol_local:VCC")
 		(at 177.8 27.94 0)
 		(unit 1)
@@
 	)
 	(symbol
-		(lib_id "PCM_SparkFun-PowerSymbol:VCC")
+		(lib_id "PCM_SparkFun-PowerSymbol_local:VCC")
 		(at 88.9 40.64 0)
 		(unit 1)
@@
 	)
 	(symbol
-		(lib_id "PCM_Diode_AKL:1N4004")
+		(lib_id "PCM_Diode_AKL_local:1N4004")
 		(at 96.52 45.72 0)
 		(unit 1)
@@
 	)
 	(symbol
-		(lib_id "PCM_SparkFun-PowerSymbol:GND")
+		(lib_id "PCM_SparkFun-PowerSymbol_local:GND")
 		(at 114.3 55.88 0)
 		(unit 1)
@@
 	)
 	(symbol
-		(lib_id "PCM_SparkFun-PowerSymbol:VIN")
+		(lib_id "PCM_SparkFun-PowerSymbol_local:VIN")
 		(at 147.32 34.29 0)
 		(unit 1)
@@
 	)
 	(symbol
-		(lib_id "PCM_SparkFun-PowerSymbol:GND")
+		(lib_id "PCM_SparkFun-PowerSymbol_local:GND")
 		(at 147.32 67.31 0)
 		(unit 1)
@@
 	)
 	(symbol
-		(lib_id "PCM_Transistor_BJT_AKL:TIP49")
+		(lib_id "PCM_Transistor_BJT_AKL_local:TIP49")
 		(at 175.26 49.53 0)
 		(unit 1)
@@
 	)
 	(symbol
-		(lib_id "PCM_SparkFun-PowerSymbol:GND")
+		(lib_id "PCM_SparkFun-PowerSymbol_local:GND")
 		(at 130.81 62.23 0)
 		(unit 1)
