File: Proyectos_KiCad/Borneras/Borneras.kicad_pcb (KiCad board)
At the start: 2 copper layers, 50 x 40 mm, 9 parts, among them J1 Screw_Terminal_01x05, J2 Screw_Terminal_01x02

Commit message: Backup antes de reinstalacion del SO: proyectos y librerias KiCad
Parts:
- added H1: ~, MountingHole:MountingHole_3.2mm_M3_Pad_Via, F.Cu at (71.5, 38.5)
- added H10: ~, MountingHole:MountingHole_3.2mm_M3_Pad_Via, F.Cu at (171.5, 67.0)
- added H11: ~, MountingHole:MountingHole_3.2mm_M3_Pad_Via, F.Cu at (131.0, 38.5)
- added H12: ~, MountingHole:MountingHole_3.2mm_M3_Pad_Via, F.Cu at (131.0, 67.0)
- added H13: ~, MountingHole:MountingHole_3.2mm_M3_Pad_Via, F.Cu at (221.5, 38.5)
- added H14: ~, MountingHole:MountingHole_3.2mm_M3_Pad_Via, F.Cu at (221.5, 67.0)
- added H15: ~, MountingHole:MountingHole_3.2mm_M3_Pad_Via, F.Cu at (181.0, 38.5)
- added H16: ~, MountingHole:MountingHole_3.2mm_M3_Pad_Via, F.Cu at (181.0, 67.0)
- added H17: ~, MountingHole:MountingHole_3.2mm_M3_Pad_Via, F.Cu at (271.5, 38.5)
- added H18: ~, MountingHole:MountingHole_3.2mm_M3_Pad_Via, F.Cu at (271.5, 67.0)
- added H19: ~, MountingHole:MountingHole_3.2mm_M3_Pad_Via, F.Cu at (231.0, 38.5)
- added H2: ~, MountingHole:MountingHole_3.2mm_M3_Pad_Via, F.Cu at (71.5, 67.0)
- added H20: ~, MountingHole:MountingHole_3.2mm_M3_Pad_Via, F.Cu at (231.0, 67.0)
- added H21: ~, MountingHole:MountingHole_3.2mm_M3_Pad_Via, F.Cu at (71.5, 78.5)
- added H22: ~, MountingHole:MountingHole_3.2mm_M3_Pad_Via, F.Cu at (71.5, 107.0)
- added H23: ~, MountingHole:MountingHole_3.2mm_M3_Pad_Via, F.Cu at (31.0, 78.5)
- added H24: ~, MountingHole:MountingHole_3.2mm_M3_Pad_Via, F.Cu at (31.0, 107.0)
- added H25: ~, MountingHole:MountingHole_3.2mm_M3_Pad_Via, F.Cu at (121.5, 78.5)
- added H26: ~, MountingHole:MountingHole_3.2mm_M3_Pad_Via, F.Cu at (121.5, 107.0)
- added H27: ~, MountingHole:MountingHole_3.2mm_M3_Pad_Via, F.Cu at (81.0, 78.5)
- added H28: ~, MountingHole:MountingHole_3.2mm_M3_Pad_Via, F.Cu at (81.0, 107.0)
- added H29: ~, MountingHole:MountingHole_3.2mm_M3_Pad_Via, F.Cu at (171.5, 78.5)
- added H3: ~, MountingHole:MountingHole_3.2mm_M3_Pad_Via, F.Cu at (31.0, 38.5)
- added H30: ~, MountingHole:MountingHole_3.2mm_M3_Pad_Via, F.Cu at (171.5, 107.0)
- added H31: ~, MountingHole:MountingHole_3.2mm_M3_Pad_Via, F.Cu at (131.0, 78.5)
- added H32: ~, MountingHole:MountingHole_3.2mm_M3_Pad_Via, F.Cu at (131.0, 107.0)
- added H33: ~, MountingHole:MountingHole_3.2mm_M3_Pad_Via, F.Cu at (221.5, 78.5)
- added H34: ~, MountingHole:MountingHole_3.2mm_M3_Pad_Via, F.Cu at (221.5, 107.0)
- added H35: ~, MountingHole:MountingHole_3.2mm_M3_Pad_Via, F.Cu at (181.0, 78.5)
- added H36: ~, MountingHole:MountingHole_3.2mm_M3_Pad_Via, F.Cu at (181.0, 107.0)
- added H4: ~, MountingHole:MountingHole_3.2mm_M3_Pad_Via, F.Cu at (31.0, 67.0)
- added H5: ~, MountingHole:MountingHole_3.2mm_M3_Pad_Via, F.Cu at (121.5, 38.5)
- added H6: ~, MountingHole:MountingHole_3.2mm_M3_Pad_Via, F.Cu at (121.5, 67.0)
- added H7: ~, MountingHole:MountingHole_3.2mm_M3_Pad_Via, F.Cu at (81.0, 38.5)
- added H8: ~, MountingHole:MountingHole_3.2mm_M3_Pad_Via, F.Cu at (81.0, 67.0)
- added H9: ~, MountingHole:MountingHole_3.2mm_M3_Pad_Via, F.Cu at (171.5, 38.5)
- added J1: Screw_Terminal_01x05, TerminalBlock_CUI:TerminalBlock_CUI_TB007-508-05_1x05_P5.08mm_Horizontal, F.Cu at (61.5, 66.5)
- added J10: Screw_Terminal_01x02, TerminalBlock_CUI:TerminalBlock_CUI_TB007-508-02_1x02_P5.08mm_Horizontal, F.Cu at (256.5, 39.5)
- added J11: Screw_Terminal_01x05, TerminalBlock_CUI:TerminalBlock_CUI_TB007-508-05_1x05_P5.08mm_Horizontal, F.Cu at (61.5, 106.5)
- added J12: Screw_Terminal_01x02, TerminalBlock_CUI:TerminalBlock_CUI_TB007-508-02_1x02_P5.08mm_Horizontal, F.Cu at (56.5, 79.5)
- added J13: Screw_Terminal_01x05, TerminalBlock_CUI:TerminalBlock_CUI_TB007-508-05_1x05_P5.08mm_Horizontal, F.Cu at (111.5, 106.5)
- added J14: Screw_Terminal_01x02, TerminalBlock_CUI:TerminalBlock_CUI_TB007-508-02_1x02_P5.08mm_Horizontal, F.Cu at (106.5, 79.5)
- added J15: Screw_Terminal_01x05, TerminalBlock_CUI:TerminalBlock_CUI_TB007-508-05_1x05_P5.08mm_Horizontal, F.Cu at (161.5, 106.5)
- added J16: Screw_Terminal_01x02, TerminalBlock_CUI:TerminalBlock_CUI_TB007-508-02_1x02_P5.08mm_Horizontal, F.Cu at (156.5, 79.5)
- added J17: Screw_Terminal_01x05, TerminalBlock_CUI:TerminalBlock_CUI_TB007-508-05_1x05_P5.08mm_Horizontal, F.Cu at (211.5, 106.5)
- added J18: Screw_Terminal_01x02, TerminalBlock_CUI:TerminalBlock_CUI_TB007-508-02_1x02_P5.08mm_Horizontal, F.Cu at (206.5, 79.5)
- added J2: Screw_Terminal_01x02, TerminalBlock_CUI:TerminalBlock_CUI_TB007-508-02_1x02_P5.08mm_Horizontal, F.Cu at (56.5, 39.5)
- added J3: Screw_Terminal_01x05, TerminalBlock_CUI:TerminalBlock_CUI_TB007-508-05_1x05_P5.08mm_Horizontal, F.Cu at (111.5, 66.5)
- added J4: Screw_Terminal_01x02, TerminalBlock_CUI:TerminalBlock_CUI_TB007-508-02_1x02_P5.08mm_Horizontal, F.Cu at (106.5, 39.5)
- added J5: Screw_Terminal_01x05, TerminalBlock_CUI:TerminalBlock_CUI_TB007-508-05_1x05_P5.08mm_Horizontal, F.Cu at (161.5, 66.5)
- added J6: Screw_Terminal_01x02, TerminalBlock_CUI:TerminalBlock_CUI_TB007-508-02_1x02_P5.08mm_Horizontal, F.Cu at (156.5, 39.5)
- added J7: Screw_Terminal_01x05, TerminalBlock_CUI:TerminalBlock_CUI_TB007-508-05_1x05_P5.08mm_Horizontal, F.Cu at (211.5, 66.5)
- added J8: Screw_Terminal_01x02, TerminalBlock_CUI:TerminalBlock_CUI_TB007-508-02_1x02_P5.08mm_Horizontal, F.Cu at (206.5, 39.5)
- added J9: Screw_Terminal_01x05, TerminalBlock_CUI:TerminalBlock_CUI_TB007-508-05_1x05_P5.08mm_Horizontal, F.Cu at (261.5, 66.5)
- added R1: 100K, Resistencias_0.25W:100K, F.Cu at (51.5, 52.5)
- added R10: 100K, Resistencias_0.25W:100K, F.Cu at (201.5, 52.5)
- added R11: 100K, Resistencias_0.25W:100K, F.Cu at (196.5, 52.5)
- added R12: 100K, Resistencias_0.25W:100K, F.Cu at (191.5, 52.5)
- added R13: 100K, Resistencias_0.25W:100K, F.Cu at (251.5, 52.5)
- added R14: 100K, Resistencias_0.25W:100K, F.Cu at (246.5, 52.5)
- added R15: 100K, Resistencias_0.25W:100K, F.Cu at (241.5, 52.5)
- added R16: 100K, Resistencias_0.25W:100K, F.Cu at (51.5, 92.5)
- added R17: 100K, Resistencias_0.25W:100K, F.Cu at (46.5, 92.5)
- added R18: 100K, Resistencias_0.25W:100K, F.Cu at (41.5, 92.5)
- added R19: 100K, Resistencias_0.25W:100K, F.Cu at (101.5, 92.5)
- added R2: 100K, Resistencias_0.25W:100K, F.Cu at (46.5, 52.5)
- added R20: 100K, Resistencias_0.25W:100K, F.Cu at (96.5, 92.5)
- added R21: 100K, Resistencias_0.25W:100K, F.Cu at (91.5, 92.5)
- added R22: 100K, Resistencias_0.25W:100K, F.Cu at (151.5, 92.5)
- added R23: 100K, Resistencias_0.25W:100K, F.Cu at (146.5, 92.5)
- added R24: 100K, Resistencias_0.25W:100K, F.Cu at (141.5, 92.5)
- added R25: 100K, Resistencias_0.25W:100K, F.Cu at (201.5, 92.5)
- added R26: 100K, Resistencias_0.25W:100K, F.Cu at (196.5, 92.5)
- added R27: 100K, Resistencias_0.25W:100K, F.Cu at (191.5, 92.5)
- added R3: 100K, Resistencias_0.25W:100K, F.Cu at (41.5, 52.5)
- added R4: 100K, Resistencias_0.25W:100K, F.Cu at (101.5, 52.5)
- added R5: 100K, Resistencias_0.25W:100K, F.Cu at (96.5, 52.5)
- added R6: 100K, Resistencias_0.25W:100K, F.Cu at (91.5, 52.5)
- added R7: 100K, Resistencias_0.25W:100K, F.Cu at (151.5, 52.5)
- added R8: 100K, Resistencias_0.25W:100K, F.Cu at (146.5, 52.5)
- added R9: 100K, Resistencias_0.25W:100K, F.Cu at (141.5, 52.5)
- moved H39 172.4 mm to (231.0, 78.5)
- moved H40 172.3 mm to (231.0, 107.0)
- moved R30 171.8 mm to (241.5, 92.5)
- moved R29 171.7 mm to (246.5, 92.5)
- moved J20 171.6 mm to (256.5, 79.5)
- moved R28 171.6 mm to (251.5, 92.5)
- moved J19 171.5 mm to (261.5, 106.5)
- moved H37 171.4 mm to (271.5, 78.5)
- moved H38 171.4 mm to (271.5, 107.0)
- renumbered H1 to H37, H2 to H38, H3 to H39, H4 to H40, J1 to J19, J2 to J20, R1 to R28, R2 to R29, R3 to R30
Routing:
- net Net-(J1-Pin_2): track 32.8 -> 327.6 mm
- net Net-(J1-Pin_1): track 27.0 -> 270.3 mm
- net Net-(J1-Pin_3): track 23.9 -> 239.2 mm
- net Net-(J1-Pin_4): track 23.9 -> 239.2 mm
- net Net-(J1-Pin_5): track 13.8 -> 138.2 mm
Other:
- board size 50 x 40 mm -> 249 x 79 mm
