File: Proyectos_KiCad/Dispenador_AguaESP32/Dispenador_AguaESP32.kicad_pcb (KiCad board)
At the start: 2 copper layers, 116.2 x 139.7 mm, 87 parts, among them J1 JACK_DC, J10 LOAD, J11 FICHERO, J2 LED12V, J3 LOAD, J4 LOAD, J5 LED12V, J6 LOAD, J7 LOAD, J8 LOAD, J9 LOAD, Q1 TIP122, Q2 BT136-800, Q3 BT136-800, Q4 TIP122, Q5 BT136-800, Q6 BT136-800, Q7 BT136-800, Q8 BT136-800, SW1 IN1, SW2 IN1, SW3 IN1, SW4 IN1, SW5 IN1, SW6 IN1, U1 MP1584, U10 74LS14, U11 ESP32_DevKit_V1_DOIT, U2 AMS1117-3.3, U3 MOC3021M, U4 MOC3021M, U5 MOC3021M, U6 MOC3021M, U7 MOC3021M, U8 MOC3021M, U9 PC817

Commit message: Guardar cambios generales
Parts:
- added H1: ~, MountingHole:MountingHole_3.2mm_M3_Pad_Via, F.Cu at (156.6, 28.8)
- added H2: ~, MountingHole:MountingHole_3.2mm_M3_Pad_Via, F.Cu at (49.9, 29.8)
- added H3: ~, MountingHole:MountingHole_3.2mm_M3_Pad_Via, F.Cu at (155.6, 164.9)
- added H4: ~, MountingHole:MountingHole_3.2mm_M3_Pad_Via, F.Cu at (48.9, 164.9)
- Q1, Q4: footprint Package_TO_SOT_THT:TO-220-3_Vertical -> @EmersonPrez15:TO-220-3_VDC
- R22, R23, R25, R27, R28, R30: footprint Resistor_SMD:R_0805_2012Metric -> Resistencias_0.25W:10K
- U12: footprint @EmersonPrez15:LCD ST7920 -> Connector_Molex:Molex_KK-254_AE-6410-04A_1x04_P2.54mm_Vertical
- U2: moved to B.Cu
- moved D9 400.7 mm to (52.5, 39.0), turned to 90 degrees
- moved J11 394.5 mm to (52.5, 50.1), turned to 90 degrees
- moved C9 381.9 mm to (65.2, 54.2), turned to 180 degrees
- moved U9 381.4 mm to (58.6, 45.1)
- moved R26 377.5 mm to (58.6, 51.2)
- moved SW6 375.3 mm to (68.2, 96.9), turned to 90 degrees
- moved R29 375.2 mm to (66.2, 37.4), turned to 180 degrees
- moved R24 371.8 mm to (66.2, 41.0), turned to 180 degrees
- moved SW5 370.0 mm to (68.2, 83.2), turned to 90 degrees
- moved SW3 369.7 mm to (52.5, 96.9), turned to 90 degrees
- moved R23 368.0 mm to (58.1, 78.1), turned to -90 degrees
- moved R25 366.2 mm to (58.1, 91.8), turned to -90 degrees
- moved SW4 364.9 mm to (68.7, 68.9), turned to 90 degrees
- moved SW2 364.4 mm to (52.5, 83.2), turned to 90 degrees
- moved R27 356.5 mm to (74.3, 63.9), turned to -90 degrees
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Connections:
- R27 pad 1: /ESP32/IN_P4 -> /ESP32/IN_P6
- R3 pad 1: /ESP32/OUT_TI1 -> /ESP32/OUT_T1
- R30 pad 1: /ESP32/IN_P6 -> /ESP32/IN_P4
- R4 pad 1: /ESP32/OUT_T1 -> /ESP32/OUT_TI2
- R9 pad 1: /ESP32/OUT_TI2 -> /ESP32/OUT_TI1
- SW4 pad 2: /ESP32/IN_P4 -> /ESP32/IN_P6
- SW6 pad 2: /ESP32/IN_P6 -> /ESP32/IN_P4
- U11 pad 17: unconnected-(U11-GND-Pad17) -> GND
Routing:
- net +12V: track 0.00 -> 265.3 mm
- net ADC1: track 0.00 -> 255.5 mm
- net +3.3V: track 0.00 -> 210.2 mm, vias 0 -> 8
- net +5V: track 0.00 -> 182.4 mm, vias 0 -> 2
- net ADC2: track 0.00 -> 157.2 mm
- net /ESP32/IN_FICHERO: track 0.00 -> 132.2 mm
- net GND: track 0.00 -> 109.6 mm, vias 0 -> 26
- net /ESP32/OUT_T1: track 0.00 -> 96.1 mm
- net /ESP32/IN_P6: track 0.00 -> 92.7 mm
- net /ESP32/OUT_T2: track 0.00 -> 89.4 mm
- net /ESP32/IN_P1: track 0.00 -> 83.5 mm
- net /ESP32/OUT_TI2: track 0.00 -> 76.3 mm
- net /ESP32/IN_P5: track 0.00 -> 75.4 mm
- net /ESP32/IN_P2: track 0.00 -> 71.8 mm
- net /ESP32/OUT_T3: track 0.00 -> 71.3 mm
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- added copper zone on B.Cu, net GND
Other:
- board size 116.2 x 139.7 mm -> 117.2 x 147.8 mm
- board text added: "12V"
- board text added: "5V"
- board text added: "GND"
- board text added: "SCL"
- board text added: "SDA"
- board text added: "SIG"
