File: Proyectos_KiCad/Dispenador_AguaESP32/ESP32.kicad_sch (KiCad schematic)
At the start: 4 parts, among them U11 ESP32_DevKit_V1_DOIT

Commit message: Guardar cambios generales
Parts:
- U12: footprint @EmersonPrez15:LCD ST7920 -> Connector_Molex:Molex_KK-254_AE-6410-04A_1x04_P2.54mm_Vertical
Connections:
- net GND: now also U11.17 (GND)
Other:
- moved on the sheet: U12
Changed lines of the file:
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@@
 	(wire
 		(pts
-			(xy 218.44 87.63) (xy 218.44 92.71)
+			(xy 218.44 78.74) (xy 218.44 92.71)
 		)
 		(stroke
@@
 	(wire
 		(pts
-			(xy 213.36 87.63) (xy 213.36 95.25)
+			(xy 213.36 78.74) (xy 213.36 95.25)
 		)
 		(stroke
@@
 	(wire
 		(pts
-			(xy 210.82 87.63) (xy 210.82 88.9)
+			(xy 210.82 78.74) (xy 210.82 88.9)
+		)
+		(stroke
+			(width 0)
+			(type default)
+		)
+	)
+	(wire
+		(pts
+			(xy 171.45 109.22) (xy 173.99 109.22)
 		)
 		(stroke
@@
 	(wire
 		(pts
-			(xy 215.9 87.63) (xy 215.9 92.71)
+			(xy 215.9 78.74) (xy 215.9 92.71)
 		)
 		(stroke
@@
 	(symbol
 		(lib_id "@EmersonPrez15:OLED_SSD1306")
-		(at 214.63 82.55 0)
+		(at 214.63 73.66 0)
 		(unit 1)
 		(body_style 1)
@@
 		(fields_autoplaced yes)
 		(property "Reference" "U12"
-			(at 220.98 78.7399 0)
+			(at 220.98 69.8499 0)
 			(show_name no)
 			(do_not_autoplace no)
@@
 		)
 		(property "Value" ""
-			(at 220.98 81.2799 0)
+			(at 220.98 72.3899 0)
 			(show_name no)
 			(do_not_autoplace no)
@@
 			)
 		)
-		(property "Footprint" "@EmersonPrez15:LCD ST7920"
-			(at 220.98 83.8199 0)
+		(property "Footprint" "Connector_Molex:Molex_KK-254_AE-6410-04A_1x04_P2.54mm_Vertical"
+			(at 220.98 74.9299 0)
 			(hide yes)
 			(show_name no)
@@
 		)
 		(property "Datasheet" ""
-			(at 214.63 82.55 0)
+			(at 214.63 73.66 0)
 			(hide yes)
 			(show_name no)
@@
 		)
 		(property "Description" ""
-			(at 214.63 82.55 0)
+			(at 214.63 73.66 0)
 			(hide yes)
 			(show_name no)
@@
 					(unit 1)
 				)
+			)
+		)
+	)
+	(symbol
+		(lib_id "power:GND")
+		(at 173.99 109.22 90)
+		(unit 1)
+		(body_style 1)
+		(exclude_from_sim no)
+		(in_bom yes)
+		(on_board yes)
+		(in_pos_files yes)
+		(dnp no)
+		(fields_autoplaced yes)
+		(property "Reference" "#PWR049"
+			(at 180.34 109.22 0)
+			(hide yes)
+			(show_name no)
+			(do_not_autoplace no)
+			(effects
+				(font
+					(size 1.27 1.27)
+				)
+			)
+		)
+		(property "Value" "GND"
+			(at 177.8 109.2199 90)
+			(show_name no)
+			(do_not_autoplace no)
+			(effects
+				(font
+					(size 1.27 1.27)
+				)
+				(justify right)
+			)
+		)
+		(property "Footprint" ""
+			(at 173.99 109.22 0)
+			(hide yes)
+			(show_name no)
+			(do_not_autoplace no)
+			(effects
+				(font
+					(size 1.27 1.27)
+				)
+			)
+		)
+		(property "Datasheet" ""
+			(at 173.99 109.22 0)
+			(hide yes)
+			(show_name no)
+			(do_not_autoplace no)
+			(effects
+				(font
+					(size 1.27 1.27)
+				)
+			)
+		)
+		(property "Description" "Power symbol creates a global label with name \"GND\" , ground"
+			(at 173.99 109.22 0)
+			(hide yes)
+			(show_name no)
+			(do_not_autoplace no)
+			(effects
+				(font
+					(size 1.27 1.27)
+				)
+			)
+		)
+		(pin "1"
+		)
+		(instances
+			(project "Dispenador_AguaESP32"
+				(path "/6715dd99-d6ac-4518-a28a-36d9343792a8/e7284cde-67e1-4185-85b4-f912288ec119"
+					(reference "#PWR049")
+					(unit 1)
+				)
