File: Proyectos_KiCad/Dispenador_AguaESP32/INPUTS.kicad_sch (KiCad schematic)
At the start: 20 parts, among them J11 FICHERO, SW1 IN1, SW2 IN1, SW3 IN1, SW4 IN1, SW5 IN1, SW6 IN1, U10 74LS14, U9 PC817

Commit message: Guardar cambios generales
Parts:
- R22, R23, R25, R27, R28, R30: footprint Resistor_SMD:R_0805_2012Metric -> Resistencias_0.25W:10K
Connections:
- net IN_P4: now also R30.1, SW6.2; no longer R27.1, SW4.2
- net IN_P6: now also R27.1, SW4.2; no longer R30.1, SW6.2
Other:
- moved on the sheet: R22, R23, R25, R27, R28, R30, SW1, SW2, SW3, SW4, SW5, SW6
