File: Proyectos_KiCad/Dispenador_AguaESP32/OUTPUTS.kicad_sch (KiCad schematic)
At the start: 55 parts, among them J10 LOAD, J2 LED12V, J3 LOAD, J4 LOAD, J5 LED12V, J6 LOAD, J7 LOAD, J8 LOAD, J9 LOAD, Q1 TIP122, Q2 BT136-800, Q3 BT136-800, Q4 TIP122, Q5 BT136-800, Q6 BT136-800, Q7 BT136-800, Q8 BT136-800, U3 MOC3021M, U4 MOC3021M, U5 MOC3021M, U6 MOC3021M, U7 MOC3021M, U8 MOC3021M

Commit message: Guardar cambios generales
Parts:
- Q1, Q4: footprint Package_TO_SOT_THT:TO-220-3_Vertical -> @EmersonPrez15:TO-220-3_VDC
Connections:
- net OUT_TI1: now also R9.1; no longer R4.1
- net OUT_TI2: now also R4.1; no longer R9.1
Changed lines of the file:
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@@
 	(wire
 		(pts
-			(xy 45.72 142.24) (xy 46.99 142.24)
+			(xy 43.18 142.24) (xy 46.99 142.24)
 		)
 		(stroke
@@
 	(wire
 		(pts
-			(xy 31.75 31.75) (xy 34.29 31.75)
+			(xy 27.94 31.75) (xy 34.29 31.75)
 		)
 		(stroke
@@
 		)
 	)
-	(hierarchical_label "OUT_TI1"
+	(hierarchical_label "OUT_TI2"
 		(shape input)
-		(at 45.72 142.24 180)
+		(at 43.18 142.24 180)
 		(effects
 			(font
@@
 	(hierarchical_label "OUT_T1"
 		(shape input)
-		(at 31.75 31.75 180)
+		(at 27.94 31.75 180)
 		(effects
 			(font
@@
 		)
 	)
-	(hierarchical_label "OUT_TI2"
+	(hierarchical_label "OUT_TI1"
 		(shape input)
 		(at 91.44 143.51 180)
@@
 			)
 		)
-		(property "Footprint" "Package_TO_SOT_THT:TO-220-3_Vertical"
+		(property "Footprint" "@EmersonPrez15:TO-220-3_VDC"
 			(at 110.49 145.415 0)
 			(hide yes)
@@
 			)
 		)
-		(property "Footprint" "Package_TO_SOT_THT:TO-220-3_Vertical"
+		(property "Footprint" "@EmersonPrez15:TO-220-3_VDC"
 			(at 64.77 144.145 0)
 			(hide yes)
