File: Proyectos_KiCad/Dispenador_AguaESP32/Power.kicad_sch (KiCad schematic)
At the start: 8 parts, among them J1 JACK_DC, U1 MP1584, U2 AMS1117-3.3

Commit message: Guardar cambios generales
Parts:
- added H1, H2, H3, H4: (no value), MountingHole:MountingHole_3.2mm_M3_Pad_Via, symbol Mechanical:MountingHole_Pad
