File: Proyectos_KiCad/Punta_Logica_CMOS/Punta_Logica_CMOS.kicad_pcb (KiCad board)
At the start: 2 copper layers, 80.5 x 25 mm, 15 parts, among them J1 VCC, U1 LM358

Commit message: Guardar cambios generales
Other:
- board text added: "9941-24-7386"
